File: DAC.sch (KiCad schematic (older format))
At the start: 21 parts

Commit message: rest of power controller
Parts:
- gave numbers to parts that had none: 21
Changed lines of the file:
@@
 $EndDescr
 $Comp
-L CS4207-CNZ:CS4207-CNZ U?
+L CS4207-CNZ:CS4207-CNZ U1
 U 1 1 5D96D6B0
 P 3600 2000
-F 0 "U?" H 5900 2388 60  0000 C CNN
+F 0 "U1" H 5900 2388 60  0000 C CNN
 F 1 "CS4207-CNZ" H 5900 2282 60  0000 C CNN
 F 2 "CIR-QFN-48_6X6" H 5900 2240 60  0001 C CNN
@@
 HDA_RESET_L
 $Comp
-L power:+1V5 #PWR?
+L power:+1V5 #PWR0101
 U 1 1 5D970ED0
 P 850 750
-F 0 "#PWR?" H 850 600 50  0001 C CNN
+F 0 "#PWR0101" H 850 600 50  0001 C CNN
 F 1 "+1V5" V 865 878 50  0000 L CNN
 F 2 "" H 850 750 50  0001 C CNN
@@
 $EndComp
 $Comp
-L pspice:INDUCTOR L?
+L pspice:INDUCTOR L1
 U 1 1 5D972FDD
 P 1350 750
-F 0 "L?" H 1350 965 50  0000 C CNN
+F 0 "L1" H 1350 965 50  0000 C CNN
 F 1 "220Ohm" H 1350 874 50  0000 C CNN
 F 2 "Inductor_SMD:L_0603_1608Metric" H 1350 750 50  0001 C CNN
@@
 $EndComp
 $Comp
-L Device:C C?
+L Device:C C1
 U 1 1 5D9737A0
 P 1800 1000
-F 0 "C?" H 1915 1046 50  0000 L CNN
+F 0 "C1" H 1915 1046 50  0000 L CNN
 F 1 "0.1uF" H 1915 955 50  0000 L CNN
 F 2 "Capacitor_SMD:C_0603_1608Metric" H 1838 850 50  0001 C CNN
@@
 $EndComp
 $Comp
-L power:GNDREF #PWR?
+L power:GNDREF #PWR0102
 U 1 1 5D97403D
 P 1800 1150
-F 0 "#PWR?" H 1800 900 50  0001 C CNN
+F 0 "#PWR0102" H 1800 900 50  0001 C CNN
 F 1 "GNDREF" H 1805 977 50  0000 C CNN
 F 2 "" H 1800 1150 50  0001 C CNN
@@
 	2800 2100 2800 2500
 $Comp
-L power:+3V3 #PWR?
+L power:+3V3 #PWR0103
 U 1 1 5D9753C1
 P 10650 950
-F 0 "#PWR?" H 10650 800 50  0001 C CNN
+F 0 "#PWR0103" H 10650 800 50  0001 C CNN
 F 1 "+3V3" V 10665 1078 50  0000 L CNN
 F 2 "" H 10650 950 50  0001 C CNN
@@
 $EndComp
 $Comp
-L Device:C C?
+L Device:C C14
 U 1 1 5D975682
 P 10450 1250
-F 0 "C?" H 10565 1296 50  0000 L CNN
+F 0 "C14" H 10565 1296 50  0000 L CNN
 F 1 "0.1uF" H 10565 1205 50  0000 L CNN
 F 2 "Capacitor_SMD:C_0603_1608Metric" H 10488 1100 50  0001 C CNN
@@
 Connection ~ 10450 950
 $Comp
-L power:GNDREF #PWR?
+L power:GNDREF #PWR0104
 U 1 1 5D976739
 P 10450 1400
-F 0 "#PWR?" H 10450 1150 50  0001 C CNN
+F 0 "#PWR0104" H 10450 1150 50  0001 C CNN
 F 1 "GNDREF" H 10455 1227 50  0000 C CNN
 F 2 "" H 10450 1400 50  0001 C CNN
@@
 $EndComp
 $Comp
-L Device:CP1 C?
+L Device:CP1 C7
 U 1 1 5D976DE3
 P 8650 1250
-F 0 "C?" H 8765 1341 50  0000 L CNN
+F 0 "C7" H 8765 1341 50  0000 L CNN
 F 1 "10uF" H 8765 1250 50  0000 L CNN
 F 2 "Capacitor_Tantalum_SMD:CP_EIA-2012-15_AVX-P" H 8650 1250 50  0001 C CNN
@@
 	8650 3800 8200 3800
 $Comp
-L Device:CP1 C?
+L Device:CP1 C10
 U 1 1 5D9788A9
 P 9750 1250
-F 0 "C?" H 9865 1341 50  0000 L CNN
+F 0 "C10" H 9865 1341 50  0000 L CNN
 F 1 "10uF" H 9865 1250 50  0000 L CNN
 F 2 "Capacitor_Tantalum_SMD:CP_EIA-2012-15_AVX-P" H 9750 1250 50  0001 C CNN
@@
 	9750 950  9750 1100
 $Comp
-L power:GNDREF #PWR?
+L power:GNDREF #PWR0105
 U 1 1 5D979064
 P 9750 1400
-F 0 "#PWR?" H 9750 1150 50  0001 C CNN
+F 0 "#PWR0105" H 9750 1150 50  0001 C CNN
 F 1 "GNDREF" H 9755 1227 50  0000 C CNN
 F 2 "" H 9750 1400 50  0001 C CNN
@@
 $EndComp
 $Comp
-L Device:C_Small C?
+L Device:C_Small C4
 U 1 1 5D979670
 P 8500 2400
-F 0 "C?" H 8592 2491 50  0000 L CNN
+F 0 "C4" H 8592 2491 50  0000 L CNN
 F 1 "2.2uF" H 8592 2400 50  0000 L CNN
 F 2 "Capacitor_SMD:C_0603_1608Metric" H 8500 2400 50  0001 C CNN
@@
 	8400 2600 8200 2600
 $Comp
-L Device:C_Small C?
+L Device:C_Small C5
 U 1 1 5D97CE57
 P 8500 2600
-F 0 "C?" H 8592 2691 50  0000 L CNN
+F 0 "C5" H 8592 2691 50  0000 L CNN
 F 1 "2.2uF" H 8592 2600 50  0000 L CNN
 F 2 "Capacitor_SMD:C_0603_1608Metric" H 8500 2600 50  0001 C CNN
@@
 $EndComp
 $Comp
-L Device:C_Small C?
+L Device:C_Small C6
 U 1 1 5D97DDD9
 P 8500 4050
-F 0 "C?" H 8592 4096 50  0000 L CNN
+F 0 "C6" H 8592 4096 50  0000 L CNN
 F 1 "1uF" H 8592 4005 50  0000 L CNN
 F 2 "Capacitor_SMD:C_0603_1608Metric" H 8500 4050 50  0001 C CNN
@@
 $EndComp
 $Comp
-L Device:C_Small C?
+L Device:C_Small C8
 U 1 1 5D97E375
 P 8800 4000
-F 0 "C?" H 8892 4046 50  0000 L CNN
+F 0 "C8" H 8892 4046 50  0000 L CNN
 F 1 "10uF" H 8892 3955 50  0000 L CNN
 F 2 "Capacitor_SMD:C_0603_1608Metric" H 8800 4000 50  0001 C CNN
@@
 Connection ~ 8500 4150
 $Comp
-L power:GNDREF #PWR?
+L power:GNDREF #PWR0106
 U 1 1 5D980EF5
 P 8500 4150
-F 0 "#PWR?" H 8500 3900 50  0001 C CNN
+F 0 "#PWR0106" H 8500 3900 50  0001 C CNN
 F 1 "GNDREF" H 8505 3977 50  0000 C CNN
 F 2 "" H 8500 4150 50  0001 C CNN
@@
 	9050 950  9050 1550
 $Comp
-L Device:C_Small C?
+L Device:C_Small C2
 U 1 1 5D9829C1
 P 2900 2900
-F 0 "C?" V 3129 2900 50  0000 C CNN
+F 0 "C2" V 3129 2900 50  0000 C CNN
 F 1 "1uF" V 3038 2900 50  0000 C CNN
 F 2 "Capacitor_SMD:C_0603_1608Metric" H 2900 2900 50  0001 C CNN
@@
 $EndComp
 $Comp
-L Device:C_Small C?
+L Device:C_Small C3
 U 1 1 5D98315B
 P 2900 3300
-F 0 "C?" V 2671 3300 50  0000 C CNN
+F 0 "C3" V 2671 3300 50  0000 C CNN
 F 1 "1uF" V 2762 3300 50  0000 C CNN
 F 2 "Capacitor_SMD:C_0603_1608Metric" H 2900 3300 50  0001 C CNN
@@
 AUD_MIC_IN_L
 $Comp
-L Device:R R?
+L Device:R R1
 U 1 1 5D98C5B8
 P 2700 3850
-F 0 "R?" H 2770 3896 50  0000 L CNN
+F 0 "R1" H 2770 3896 50  0000 L CNN
 F 1 "2.2kOhm" H 2770 3805 50  0000 L CNN
 F 2 "Resistor_SMD:R_0603_1608Metric" V 2630 3850 50  0001 C CNN
@@
 $EndComp
 $Comp
-L Device:R R?
+L Device:R R2
 U 1 1 5D98C630
 P 3200 3850
-F 0 "R?" H 3270 3896 50  0000 L CNN
+F 0 "R2" H 3270 3896 50  0000 L CNN
 F 1 "2.2kOhm" H 3270 3805 50  0000 L CNN
 F 2 "Resistor_SMD:R_0603_1608Metric" V 3130 3850 50  0001 C CNN
@@
 	8400 2700 8500 2700
 $Comp
-L Device:C C?
+L Device:C C11
 U 1 1 5D997154
 P 9900 2600
-F 0 "C?" H 10015 2646 50  0000 L CNN
+F 0 "C11" H 10015 2646 50  0000 L CNN
 F 1 "0.1uF" H 10015 2555 50  0000 L CNN
 F 2 "Capacitor_SMD:C_0603_1608Metric" H 9938 2450 50  0001 C CNN
@@
 	9900 2900 9900 2950
 $Comp
-L Device:R R?
+L Device:R R4
 U 1 1 5D99A829
 P 9750 3250
-F 0 "R?" V 9543 3250 50  0000 C CNN
+F 0 "R4" V 9543 3250 50  0000 C CNN
 F 1 "33Ohm" V 9634 3250 50  0000 C CNN
 F 2 "Resistor_SMD:R_0603_1608Metric" V 9680 3250 50  0001 C CNN
@@
 $EndComp
 $Comp
-L Device:R R?
+L Device:R R3
 U 1 1 5D99AF4D
 P 9750 2450
-F 0 "R?" V 9543 2450 50  0000 C CNN
+F 0 "R3" V 9543 2450 50  0000 C CNN
 F 1 "33Ohm" V 9634 2450 50  0000 C CNN
 F 2 "Resistor_SMD:R_0603_1608Metric" V 9680 2450 50  0001 C CNN
@@
 $EndComp
 $Comp
-L power:GNDREF #PWR?
+L power:GNDREF #PWR0107
 U 1 1 5D99B4F2
 P 9600 2450
-F 0 "#PWR?" H 9600 2200 50  0001 C CNN
+F 0 "#PWR0107" H 9600 2200 50  0001 C CNN
 F 1 "GNDREF" V 9605 2322 50  0000 R CNN
 F 2 "" H 9600 2450 50  0001 C CNN
@@
 $EndComp
 $Comp
-L power:GNDREF #PWR?
+L power:GNDREF #PWR0108
 U 1 1 5D99BC64
 P 9600 3250
-F 0 "#PWR?" H 9600 3000 50  0001 C CNN
+F 0 "#PWR0108" H 9600 3000 50  0001 C CNN
 F 1 "GNDREF" V 9605 3122 50  0000 R CNN
 F 2 "" H 9600 3250 50  0001 C CNN
@@
 $EndComp
 $Comp
-L Device:C C?
+L Device:C C12
 U 1 1 5D99C508
 P 9900 3100
-F 0 "C?" H 10015 3146 50  0000 L CNN
+F 0 "C12" H 10015 3146 50  0000 L CNN
 F 1 "0.1uF" H 10015 3055 50  0000 L CNN
 F 2 "Capacitor_SMD:C_0603_1608Metric" H 9938 2950 50  0001 C CNN
@@
 Connection ~ 9900 2900
 $Comp
-L power:GNDREF #PWR?
+L power:GNDREF #PWR0109
 U 1 1 5D9A0E0C
 P 3400 3650
-F 0 "#PWR?" H 3400 3400 50  0001 C CNN
+F 0 "#PWR0109" H 3400 3400 50  0001 C CNN
 F 1 "GNDREF" H 3405 3477 50  0000 C CNN
 F 2 "" H 3400 3650 50  0001 C CNN
@@
 Connection ~ 9050 1550
 $Comp
-L Device:C_Small C?
+L Device:C_Small C9
 U 1 1 5D9AE73B
 P 9600 3850
-F 0 "C?" H 9692 3896 50  0000 L CNN
+F 0 "C9" H 9692 3896 50  0000 L CNN
 F 1 "0.1uF" H 9692 3805 50  0000 L CNN
 F 2 "Capacitor_SMD:C_0603_1608Metric" H 9600 3850 50  0001 C CNN
@@
 $EndComp
 $Comp
-L Device:C_Small C?
+L Device:C_Small C13
 U 1 1 5D9AEC18
 P 10050 3850
-F 0 "C?" H 10142 3941 50  0000 L CNN
+F 0 "C13" H 10142 3941 50  0000 L CNN
 F 1 "10uF" H 10142 3850 50  0000 L CNN
 F 2 "Capacitor_SMD:C_0603_1608Metric" H 10050 3850 50  0001 C CNN
@@
 $EndComp
 $Comp
-L power:GNDREF #PWR?
+L power:GNDREF #PWR0110
 U 1 1 5D9AF888
 P 10500 4200
-F 0 "#PWR?" H 10500 3950 50  0001 C CNN
+F 0 "#PWR0110" H 10500 3950 50  0001 C CNN
 F 1 "GNDREF" H 10505 4027 50  0000 C CNN
 F 2 "" H 10500 4200 50  0001 C CNN
@@
 	10500 3700 10500 3750
 $Comp
-L Device:C_Small C?
+L Device:C_Small C15
 U 1 1 5D9BEAD3
 P 10500 3850
-F 0 "C?" H 10592 3941 50  0000 L CNN
+F 0 "C15" H 10592 3941 50  0000 L CNN
 F 1 "10uF" H 10592 3850 50  0000 L CNN
 F 2 "Capacitor_SMD:C_0603_1608Metric" H 10500 3850 50  0001 C CNN
