File: DAC.sch (KiCad schematic (older format))
At the start: 21 parts, among them U1 CS4207-CNZ

Commit message: Finished all except RAM and CPU
Parts:
- U1: footprint CIR-QFN-48_6X6 -> CS4207-CNZ:CS4207-CNZ
Changed lines of the file:
@@
 $Descr A4 11693 8268
 encoding utf-8
-Sheet 2 23
+Sheet 2 24
 Title ""
 Date ""
@@
 F 0 "U1" H 5900 2388 60  0000 C CNN
 F 1 "CS4207-CNZ" H 5900 2282 60  0000 C CNN
-F 2 "CIR-QFN-48_6X6" H 5900 2240 60  0001 C CNN
+F 2 "CS4207-CNZ:CS4207-CNZ" H 5900 2240 60  0001 C CNN
 F 3 "" H 3600 2000 60  0000 C CNN
 	1    3600 2000
