File: HDMI.sch (KiCad schematic (older format))
At the start: 16 parts

Commit message: finishing schematic
Parts:
- gave numbers to parts that had none: 16
Changed lines of the file:
@@
 $Descr A4 11693 8268
 encoding utf-8
-Sheet 4 20
+Sheet 4 21
 Title ""
 Date ""
@@
 $EndDescr
 $Comp
-L TPD12S016PW:TPD12S016PWR U?
+L TPD12S016PW:TPD12S016PWR U3
 U 1 1 5DA7626E
 P 5500 4650
-F 0 "U?" H 6900 5037 60  0000 C CNN
+F 0 "U3" H 6900 5037 60  0000 C CNN
 F 1 "TPD12S016PWR" H 6900 4931 60  0000 C CNN
 F 2 "PW24" H 6900 4890 60  0001 C CNN
@@
 $EndComp
 $Comp
-L Connector:HDMI_A J?
+L Connector:HDMI_A J1
 U 1 1 5DA77FC3
 P 9300 3050
-F 0 "J?" H 9730 3096 50  0000 L CNN
+F 0 "J1" H 9730 3096 50  0000 L CNN
 F 1 "HDMI_A" H 9730 3005 50  0000 L CNN
 F 2 "" H 9325 3050 50  0001 C CNN
@@
 	8900 3750 5500 3750
 $Comp
-L power:GND #PWR?
+L power:GND #PWR0143
 U 1 1 5DA7EE5E
 P 9100 4600
-F 0 "#PWR?" H 9100 4350 50  0001 C CNN
+F 0 "#PWR0143" H 9100 4350 50  0001 C CNN
 F 1 "GND" H 9105 4427 50  0000 C CNN
 F 2 "" H 9100 4600 50  0001 C CNN
@@
 Connection ~ 9500 4250
 $Comp
-L Device:R_Small R?
+L Device:R_Small R63
 U 1 1 5DA8114D
 P 5200 1450
-F 0 "R?" H 5259 1496 50  0000 L CNN
+F 0 "R63" H 5259 1496 50  0000 L CNN
 F 1 "10KOhm" H 5259 1405 50  0000 L CNN
 F 2 "" H 5200 1450 50  0001 C CNN
@@
 $EndComp
 $Comp
-L Device:R_Small R?
+L Device:R_Small R64
 U 1 1 5DA811CD
 P 5400 1450
-F 0 "R?" H 5459 1496 50  0000 L CNN
+F 0 "R64" H 5459 1496 50  0000 L CNN
 F 1 "10KOhm" H 5459 1405 50  0000 L CNN
 F 2 "" H 5400 1450 50  0001 C CNN
@@
 $EndComp
 $Comp
-L Device:R_Small R?
+L Device:R_Small R62
 U 1 1 5DA813B9
 P 4700 1100
-F 0 "R?" H 4759 1146 50  0000 L CNN
+F 0 "R62" H 4759 1146 50  0000 L CNN
 F 1 "2.2KOkm" H 4759 1055 50  0000 L CNN
 F 2 "" H 4700 1100 50  0001 C CNN
@@
 $EndComp
 $Comp
-L Device:R_Small R?
+L Device:R_Small R61
 U 1 1 5DA81A04
 P 4550 1100
-F 0 "R?" H 4609 1146 50  0000 L CNN
+F 0 "R61" H 4609 1146 50  0000 L CNN
 F 1 "2.2KOhm" H 4609 1055 50  0000 L CNN
 F 2 "" H 4550 1100 50  0001 C CNN
@@
 $EndComp
 $Comp
-L Device:R_Small R?
+L Device:R_Small R59
 U 1 1 5DA81C54
 P 3450 1450
-F 0 "R?" V 3254 1450 50  0000 C CNN
+F 0 "R59" V 3254 1450 50  0000 C CNN
 F 1 "0Ohm" V 3345 1450 50  0000 C CNN
 F 2 "" H 3450 1450 50  0001 C CNN
@@
 $EndComp
 $Comp
-L Device:R_Small R?
+L Device:R_Small R60
 U 1 1 5DA8221D
 P 3450 1600
-F 0 "R?" V 3254 1600 50  0000 C CNN
+F 0 "R60" V 3254 1600 50  0000 C CNN
 F 1 "0Ohm" V 3345 1600 50  0000 C CNN
 F 2 "" H 3450 1600 50  0001 C CNN
@@
 $EndComp
 $Comp
-L Device:R_Small R?
+L Device:R_Small R67
 U 1 1 5DA824EC
 P 6050 4350
-F 0 "R?" V 5854 4350 50  0000 C CNN
+F 0 "R67" V 5854 4350 50  0000 C CNN
 F 1 "0Ohm" V 5945 4350 50  0000 C CNN
 F 2 "" H 6050 4350 50  0001 C CNN
@@
 	5900 3450 5900 3850
 $Comp
-L Device:R_Small R?
+L Device:R_Small R69
 U 1 1 5DA8514F
 P 7100 1300
-F 0 "R?" H 7159 1346 50  0000 L CNN
+F 0 "R69" H 7159 1346 50  0000 L CNN
 F 1 "100KOhm" H 7159 1255 50  0000 L CNN
 F 2 "" H 7100 1300 50  0001 C CNN
@@
 	7100 1200 7550 1200
 $Comp
-L Device:C_Small C?
+L Device:C_Small C51
 U 1 1 5DA85C5F
 P 7550 1300
-F 0 "C?" H 7642 1346 50  0000 L CNN
+F 0 "C51" H 7642 1346 50  0000 L CNN
 F 1 "4.7uF" H 7642 1255 50  0000 L CNN
 F 2 "" H 7550 1300 50  0001 C CNN
@@
 $EndComp
 $Comp
-L power:GND #PWR?
+L power:GND #PWR0144
 U 1 1 5DA86343
 P 7100 1400
-F 0 "#PWR?" H 7100 1150 50  0001 C CNN
+F 0 "#PWR0144" H 7100 1150 50  0001 C CNN
 F 1 "GND" H 7105 1227 50  0000 C CNN
 F 2 "" H 7100 1400 50  0001 C CNN
@@
 $EndComp
 $Comp
-L power:GND #PWR?
+L power:GND #PWR0145
 U 1 1 5DA863A5
 P 7550 1400
-F 0 "#PWR?" H 7550 1150 50  0001 C CNN
+F 0 "#PWR0145" H 7550 1150 50  0001 C CNN
 F 1 "GND" H 7555 1227 50  0000 C CNN
 F 2 "" H 7550 1400 50  0001 C CNN
@@
 $EndComp
 $Comp
-L pspice:INDUCTOR L?
+L pspice:INDUCTOR L2
 U 1 1 5DA8688A
 P 7350 1850
-F 0 "L?" H 7350 2065 50  0000 C CNN
+F 0 "L2" H 7350 2065 50  0000 C CNN
 F 1 "FB_220R_2.2A" H 7350 1974 50  0000 C CNN
 F 2 "" H 7350 1850 50  0001 C CNN
@@
 $EndComp
 $Comp
-L power:GND #PWR?
+L power:GND #PWR0146
 U 1 1 5DA883D2
 P 2700 3650
-F 0 "#PWR?" H 2700 3400 50  0001 C CNN
+F 0 "#PWR0146" H 2700 3400 50  0001 C CNN
 F 1 "GND" V 2705 3522 50  0000 R CNN
 F 2 "" H 2700 3650 50  0001 C CNN
@@
 $EndComp
 $Comp
-L power:GND #PWR?
+L power:GND #PWR0147
 U 1 1 5DA887A6
 P 2700 4150
-F 0 "#PWR?" H 2700 3900 50  0001 C CNN
+F 0 "#PWR0147" H 2700 3900 50  0001 C CNN
 F 1 "GND" V 2705 4022 50  0000 R CNN
 F 2 "" H 2700 4150 50  0001 C CNN
@@
 $EndComp
 $Comp
-L power:GND #PWR?
+L power:GND #PWR0148
 U 1 1 5DA88BD3
 P 5500 4150
-F 0 "#PWR?" H 5500 3900 50  0001 C CNN
+F 0 "#PWR0148" H 5500 3900 50  0001 C CNN
 F 1 "GND" V 5505 4022 50  0000 R CNN
 F 2 "" H 5500 4150 50  0001 C CNN
@@
 	5400 1200 6150 1200
 $Comp
-L POWER:+HDMI_CRT_VCC #PWR?
+L POWER:+HDMI_CRT_VCC #PWR0149
 U 1 1 5DA982C9
 P 5400 900
-F 0 "#PWR?" H 5400 750 50  0001 C CNN
+F 0 "#PWR0149" H 5400 750 50  0001 C CNN
 F 1 "+HDMI_CRT_VCC" H 5417 1073 50  0000 C CNN
 F 2 "" H 5400 900 50  0001 C CNN
@@
 	5400 900  5400 1200
 $Comp
-L POWER:+V1P8S #PWR?
+L POWER:+V1P8S #PWR0150
 U 1 1 5DA9B64E
 P 4700 900
-F 0 "#PWR?" H 4700 750 50  0001 C CNN
+F 0 "#PWR0150" H 4700 750 50  0001 C CNN
 F 1 "+V1P8S" H 4717 1073 50  0000 C CNN
 F 2 "" H 4700 900 50  0001 C CNN
@@
 	9300 1850 9300 1950
 $Comp
-L Device:C_Small C?
+L Device:C_Small C50
 U 1 1 5DAA95E7
 P 2550 4850
-F 0 "C?" H 2642 4896 50  0000 L CNN
+F 0 "C50" H 2642 4896 50  0000 L CNN
 F 1 "0.1uF" H 2642 4805 50  0000 L CNN
 F 2 "" H 2550 4850 50  0001 C CNN
@@
 $EndComp
 $Comp
-L power:GND #PWR?
+L power:GND #PWR0151
 U 1 1 5DAAA2C6
 P 2550 4950
-F 0 "#PWR?" H 2550 4700 50  0001 C CNN
+F 0 "#PWR0151" H 2550 4700 50  0001 C CNN
 F 1 "GND" H 2555 4777 50  0000 C CNN
 F 2 "" H 2550 4950 50  0001 C CNN
@@
 	2550 4650 2550 4750
 $Comp
-L POWER:+V1P8S #PWR?
+L POWER:+V1P8S #PWR0152
 U 1 1 5DAABC22
 P 2300 4650
-F 0 "#PWR?" H 2300 4500 50  0001 C CNN
+F 0 "#PWR0152" H 2300 4500 50  0001 C CNN
 F 1 "+V1P8S" V 2318 4778 50  0000 L CNN
 F 2 "" H 2300 4650 50  0001 C CNN
@@
 Connection ~ 2550 4650
 $Comp
-L POWER:+V1P8S #PWR?
+L POWER:+V1P8S #PWR0153
 U 1 1 5DAADF43
 P 5850 5350
-F 0 "#PWR?" H 5850 5200 50  0001 C CNN
+F 0 "#PWR0153" H 5850 5200 50  0001 C CNN
 F 1 "+V1P8S" H 5868 5523 50  0000 C CNN
 F 2 "" H 5850 5350 50  0001 C CNN
@@
 $EndComp
 $Comp
-L Device:R_Small R?
+L Device:R_Small R65
 U 1 1 5DAADFF7
 P 5850 5000
-F 0 "R?" H 5909 5046 50  0000 L CNN
+F 0 "R65" H 5909 5046 50  0000 L CNN
 F 1 "10KOhm" H 5909 4955 50  0000 L CNN
 F 2 "" H 5850 5000 50  0001 C CNN
@@
 $EndComp
 $Comp
-L Device:R_Small R?
+L Device:R_Small R66
 U 1 1 5DAAE788
 P 6000 5000
-F 0 "R?" H 6059 5046 50  0000 L CNN
+F 0 "R66" H 6059 5046 50  0000 L CNN
 F 1 "10KOhm" H 6059 4955 50  0000 L CNN
 F 2 "" H 6000 5000 50  0001 C CNN
@@
 $EndComp
 $Comp
-L Device:R_Small R?
+L Device:R_Small R68
 U 1 1 5DAAEA17
 P 6150 5000
-F 0 "R?" H 6209 5046 50  0000 L CNN
+F 0 "R68" H 6209 5046 50  0000 L CNN
 F 1 "10KOhm" H 6209 4955 50  0000 L CNN
 F 2 "" H 6150 5000 50  0001 C CNN

Commit message: Finished all except RAM and CPU
Parts:
- C50, C51: footprint (none) -> Capacitor_SMD:C_0603_1608Metric
- J1: value HDMI_A -> 10029449-111RLF; footprint (none) -> 10029449-111RLF:10029449-111RLF
- L2: footprint (none) -> Inductor_SMD:L_0603_1608Metric
- R59, R60, R61, R62, R63, R64, R65, R66, R67, R68, R69: footprint (none) -> Resistor_SMD:R_0603_1608Metric
- U3: footprint PW24 -> TPD12S016PW:TPD12S016PWR
Changed lines of the file:
@@
 $Descr A4 11693 8268
 encoding utf-8
-Sheet 4 23
+Sheet 4 24
 Title ""
 Date ""
@@
 F 0 "U3" H 6900 5037 60  0000 C CNN
 F 1 "TPD12S016PWR" H 6900 4931 60  0000 C CNN
-F 2 "PW24" H 6900 4890 60  0001 C CNN
+F 2 "TPD12S016PW:TPD12S016PWR" H 6900 4890 60  0001 C CNN
 F 3 "" H 5500 4650 60  0000 C CNN
 	1    5500 4650
@@
 P 9300 3050
 F 0 "J1" H 9730 3096 50  0000 L CNN
-F 1 "HDMI_A" H 9730 3005 50  0000 L CNN
-F 2 "" H 9325 3050 50  0001 C CNN
+F 1 "10029449-111RLF" H 9730 3005 50  0000 L CNN
+F 2 "10029449-111RLF:10029449-111RLF" H 9325 3050 50  0001 C CNN
 F 3 "https://en.wikipedia.org/wiki/HDMI" H 9325 3050 50  0001 C CNN
 	1    9300 3050
@@
 F 0 "R63" H 5259 1496 50  0000 L CNN
 F 1 "10KOhm" H 5259 1405 50  0000 L CNN
-F 2 "" H 5200 1450 50  0001 C CNN
+F 2 "Resistor_SMD:R_0603_1608Metric" H 5200 1450 50  0001 C CNN
 F 3 "~" H 5200 1450 50  0001 C CNN
 	1    5200 1450
@@
 F 0 "R64" H 5459 1496 50  0000 L CNN
 F 1 "10KOhm" H 5459 1405 50  0000 L CNN
-F 2 "" H 5400 1450 50  0001 C CNN
+F 2 "Resistor_SMD:R_0603_1608Metric" H 5400 1450 50  0001 C CNN
 F 3 "~" H 5400 1450 50  0001 C CNN
 	1    5400 1450
@@
 F 0 "R62" H 4759 1146 50  0000 L CNN
 F 1 "2.2KOkm" H 4759 1055 50  0000 L CNN
-F 2 "" H 4700 1100 50  0001 C CNN
+F 2 "Resistor_SMD:R_0603_1608Metric" H 4700 1100 50  0001 C CNN
 F 3 "~" H 4700 1100 50  0001 C CNN
 	1    4700 1100
@@
 F 0 "R61" H 4609 1146 50  0000 L CNN
 F 1 "2.2KOhm" H 4609 1055 50  0000 L CNN
-F 2 "" H 4550 1100 50  0001 C CNN
+F 2 "Resistor_SMD:R_0603_1608Metric" H 4550 1100 50  0001 C CNN
 F 3 "~" H 4550 1100 50  0001 C CNN
 	1    4550 1100
@@
 F 0 "R59" V 3254 1450 50  0000 C CNN
 F 1 "0Ohm" V 3345 1450 50  0000 C CNN
-F 2 "" H 3450 1450 50  0001 C CNN
+F 2 "Resistor_SMD:R_0603_1608Metric" H 3450 1450 50  0001 C CNN
 F 3 "~" H 3450 1450 50  0001 C CNN
 	1    3450 1450
@@
 F 0 "R60" V 3254 1600 50  0000 C CNN
 F 1 "0Ohm" V 3345 1600 50  0000 C CNN
-F 2 "" H 3450 1600 50  0001 C CNN
+F 2 "Resistor_SMD:R_0603_1608Metric" H 3450 1600 50  0001 C CNN
 F 3 "~" H 3450 1600 50  0001 C CNN
 	1    3450 1600
@@
 F 0 "R67" V 5854 4350 50  0000 C CNN
 F 1 "0Ohm" V 5945 4350 50  0000 C CNN
-F 2 "" H 6050 4350 50  0001 C CNN
+F 2 "Resistor_SMD:R_0603_1608Metric" H 6050 4350 50  0001 C CNN
 F 3 "~" H 6050 4350 50  0001 C CNN
 	1    6050 4350
@@
 F 0 "R69" H 7159 1346 50  0000 L CNN
 F 1 "100KOhm" H 7159 1255 50  0000 L CNN
-F 2 "" H 7100 1300 50  0001 C CNN
+F 2 "Resistor_SMD:R_0603_1608Metric" H 7100 1300 50  0001 C CNN
 F 3 "~" H 7100 1300 50  0001 C CNN
 	1    7100 1300
@@
 F 0 "C51" H 7642 1346 50  0000 L CNN
 F 1 "4.7uF" H 7642 1255 50  0000 L CNN
-F 2 "" H 7550 1300 50  0001 C CNN
+F 2 "Capacitor_SMD:C_0603_1608Metric" H 7550 1300 50  0001 C CNN
 F 3 "~" H 7550 1300 50  0001 C CNN
 	1    7550 1300
@@
 F 0 "L2" H 7350 2065 50  0000 C CNN
 F 1 "FB_220R_2.2A" H 7350 1974 50  0000 C CNN
-F 2 "" H 7350 1850 50  0001 C CNN
+F 2 "Inductor_SMD:L_0603_1608Metric" H 7350 1850 50  0001 C CNN
 F 3 "~" H 7350 1850 50  0001 C CNN
 	1    7350 1850
@@
 F 0 "C50" H 2642 4896 50  0000 L CNN
 F 1 "0.1uF" H 2642 4805 50  0000 L CNN
-F 2 "" H 2550 4850 50  0001 C CNN
+F 2 "Capacitor_SMD:C_0603_1608Metric" H 2550 4850 50  0001 C CNN
 F 3 "~" H 2550 4850 50  0001 C CNN
 	1    2550 4850
@@
 F 0 "R65" H 5909 5046 50  0000 L CNN
 F 1 "10KOhm" H 5909 4955 50  0000 L CNN
-F 2 "" H 5850 5000 50  0001 C CNN
+F 2 "Resistor_SMD:R_0603_1608Metric" H 5850 5000 50  0001 C CNN
 F 3 "~" H 5850 5000 50  0001 C CNN
 	1    5850 5000
@@
 F 0 "R66" H 6059 5046 50  0000 L CNN
 F 1 "10KOhm" H 6059 4955 50  0000 L CNN
-F 2 "" H 6000 5000 50  0001 C CNN
+F 2 "Resistor_SMD:R_0603_1608Metric" H 6000 5000 50  0001 C CNN
 F 3 "~" H 6000 5000 50  0001 C CNN
 	1    6000 5000
@@
 F 0 "R68" H 6209 5046 50  0000 L CNN
 F 1 "10KOhm" H 6209 4955 50  0000 L CNN
-F 2 "" H 6150 5000 50  0001 C CNN
+F 2 "Resistor_SMD:R_0603_1608Metric" H 6150 5000 50  0001 C CNN
 F 3 "~" H 6150 5000 50  0001 C CNN
 	1    6150 5000
