File: MEM.sch (KiCad schematic (older format))
At the start: 0 parts

Commit message: split cpu and created more power schema
Parts:
- added J? (x2): SODIMM-200, symbol Connector:SODIMM-200
Changed lines of the file:
@@
 $Descr A4 11693 8268
 encoding utf-8
-Sheet 1 7
+Sheet 6 20
 Title ""
 Date ""
@@
 Comment4 ""
 $EndDescr
+$Comp
+L Connector:SODIMM-200 J?
+U 1 1 5DB94EE7
+P 9100 3400
+F 0 "J?" H 9100 4565 50  0000 C CNN
+F 1 "SODIMM-200" H 9100 4474 50  0000 C CNN
+F 2 "" H 10500 7250 50  0001 C CNN
+F 3 "~" H 10500 7250 50  0001 C CNN
+	1    9100 3400
+	1    0    0    -1
+$EndComp
+$Comp
+L Connector:SODIMM-200 J?
+U 2 1 5DB9FF88
+P 3650 4100
+F 0 "J?" H 3650 8265 50  0000 C CNN
+F 1 "SODIMM-200" H 3650 8174 50  0000 C CNN
+F 2 "" H 5050 7950 50  0001 C CNN
+F 3 "~" H 5050 7950 50  0001 C CNN
+	2    3650 4100
+	1    0    0    -1
+$EndComp
 $EndSCHEMATC

Commit message: finishing schematic
Parts:
- gave numbers to parts that had none: 1
Changed lines of the file:
@@
 $Descr A4 11693 8268
 encoding utf-8
-Sheet 6 20
+Sheet 6 21
 Title ""
 Date ""
@@
 $EndDescr
 $Comp
-L Connector:SODIMM-200 J?
+L Connector:SODIMM-200 J4
 U 1 1 5DB94EE7
 P 9100 3400
-F 0 "J?" H 9100 4565 50  0000 C CNN
+F 0 "J4" H 9100 4565 50  0000 C CNN
 F 1 "SODIMM-200" H 9100 4474 50  0000 C CNN
 F 2 "" H 10500 7250 50  0001 C CNN
@@
 $EndComp
 $Comp
-L Connector:SODIMM-200 J?
+L Connector:SODIMM-200 J4
 U 2 1 5DB9FF88
 P 3650 4100
-F 0 "J?" H 3650 8265 50  0000 C CNN
+F 0 "J4" H 3650 8265 50  0000 C CNN
 F 1 "SODIMM-200" H 3650 8174 50  0000 C CNN
 F 2 "" H 5050 7950 50  0001 C CNN

Commit message: Finished all except RAM and CPU
Parts:
- J4: footprint (none) -> 2013289-1:2013289-1
Changed lines of the file:
@@
 $Descr A4 11693 8268
 encoding utf-8
-Sheet 6 23
+Sheet 6 24
 Title ""
 Date ""
@@
 F 0 "J4" H 9100 4565 50  0000 C CNN
 F 1 "SODIMM-200" H 9100 4474 50  0000 C CNN
-F 2 "" H 10500 7250 50  0001 C CNN
+F 2 "2013289-1:2013289-1" H 10500 7250 50  0001 C CNN
 F 3 "~" H 10500 7250 50  0001 C CNN
 	1    9100 3400
@@
 F 0 "J4" H 3650 8265 50  0000 C CNN
 F 1 "SODIMM-200" H 3650 8174 50  0000 C CNN
-F 2 "" H 5050 7950 50  0001 C CNN
+F 2 "2013289-1:2013289-1" H 5050 7950 50  0001 C CNN
 F 3 "~" H 5050 7950 50  0001 C CNN
 	2    3650 4100
