File: PD2.sch (KiCad schematic (older format))
At the start: 45 parts

Commit message: finishing schematic
Parts:
- added C95: 0.1uF, Capacitor_SMD:C_0603_1608Metric, symbol Device:C_Small
- added R88: 33Ohm, Resistor_SMD:R_0603_1608Metric, symbol Device:R_Small
- added R89: 2.2KOhm, Resistor_SMD:R_0603_1608Metric, symbol Device:R_Small
- added R90, R91: 1KOhm, Resistor_SMD:R_0603_1608Metric, symbol Device:R_Small
- added U23: NCT3012S, symbol NCT3012S:NCT3012S
- gave numbers to parts that had none: 45
Connections:
- net +PS_3VSB: now also R91.2
- net +PS_5VSB: now also C95.1, R89.2, R90.2, U23.2 (VSB)
- net GND: now also C95.2
- new net: R89.1, U23.1 (DeepS5_Sel)
- new net: R88.1, U23.3 (PS_IN#)
- new net 5VSB_CTRL: R90.1, U23.8 (SYS5VSB_OFF)
- new net DDR_SMB_CLK: U23.6 (SCLK)
- new net DDR_SMB_DATA: U23.5 (SDA)
- new net FP_PWRBTN: R88.2
- new net PS_OUT_L: R91.1, U23.7 (PS_OUT#)
- new net SLP_S4_L: U23.4 (SLP_S5#)

Commit message: Finished all except RAM and CPU
Parts:
- J6: footprint (none) -> Connector_BarrelJack:BarrelJack_Horizontal
- L11, L12, L13, L14: footprint (none) -> Inductor_SMD:L_0603_1608Metric
- U21: footprint (none) -> cust:VQFN_EP
- U22: footprint (none) -> Package_SO:SO-8_5.3x6.2mm_P1.27mm
- U23: footprint (none) -> Package_SO:SOIC-8_3.9x4.9mm_P1.27mm
Changed lines of the file:
@@
 $Descr A4 11693 8268
 encoding utf-8
-Sheet 20 23
+Sheet 20 24
 Title ""
 Date ""
@@
 F 0 "J6" H 938 946 50  0000 L CNN
 F 1 "Conn_Coaxial_Power" H 938 855 50  0000 L CNN
-F 2 "" H 850 900 50  0001 C CNN
+F 2 "Connector_BarrelJack:BarrelJack_Horizontal" H 850 900 50  0001 C CNN
 F 3 "~" H 850 900 50  0001 C CNN
 	1    850  950
@@
 F 0 "U22" H 4100 1790 60  0000 C CNN
 F 1 "IRF9321" H 4100 1684 60  0000 C CNN
-F 2 "" H 3800 1550 60  0001 L CNN
+F 2 "Package_SO:SO-8_5.3x6.2mm_P1.27mm" H 3800 1550 60  0001 L CNN
 F 3 "" H 3800 1350 60  0001 L CNN
 	1    3600 1500
@@
 F 0 "L13" V 2446 1256 50  0000 R CNN
 F 1 "FB_120R_3A" V 2355 1256 50  0000 R CNN
-F 2 "" H 2400 1300 50  0001 C CNN
+F 2 "Inductor_SMD:L_0603_1608Metric" H 2400 1300 50  0001 C CNN
 F 3 "~" H 2400 1300 50  0001 C CNN
 	1    2400 1300
@@
 F 0 "L14" V 2696 1256 50  0000 R CNN
 F 1 "FB_120R_3A" V 2605 1256 50  0000 R CNN
-F 2 "" H 2650 1300 50  0001 C CNN
+F 2 "Inductor_SMD:L_0603_1608Metric" H 2650 1300 50  0001 C CNN
 F 3 "~" H 2650 1300 50  0001 C CNN
 	1    2650 1300
@@
 F 0 "U21" H 3250 5703 60  0000 C CNN
 F 1 "NB670" H 3250 5597 60  0000 C CNN
-F 2 "" H 2600 4950 60  0001 R CNN
+F 2 "cust:VQFN_EP" H 2600 4950 60  0001 R CNN
 F 3 "" H 2600 4750 60  0001 R CNN
 	1    2450 4900
@@
 F 0 "L11" V 996 4156 50  0000 R CNN
 F 1 "FB_120R_3A" V 905 4156 50  0000 R CNN
-F 2 "" H 950 4200 50  0001 C CNN
+F 2 "Inductor_SMD:L_0603_1608Metric" H 950 4200 50  0001 C CNN
 F 3 "~" H 950 4200 50  0001 C CNN
 	1    950  4200
@@
 F 0 "L12" V 996 4256 50  0000 R CNN
 F 1 "FB_120R_3A" V 905 4256 50  0000 R CNN
-F 2 "" H 950 4300 50  0001 C CNN
+F 2 "Inductor_SMD:L_0603_1608Metric" H 950 4300 50  0001 C CNN
 F 3 "~" H 950 4300 50  0001 C CNN
 	1    950  4300
@@
 F 0 "U23" H 8750 1840 60  0000 C CNN
 F 1 "NCT3012S" H 8750 1734 60  0000 C CNN
-F 2 "" H 8100 1600 60  0001 L CNN
+F 2 "Package_SO:SOIC-8_3.9x4.9mm_P1.27mm" H 8100 1600 60  0001 L CNN
 F 3 "" H 8100 1400 60  0001 L CNN
 	1    7900 1550
