File: PD3.sch (KiCad schematic (older format))
At the start: 27 parts, among them Q1 2N7002K, Q2 2N7002K, Q3 MMBT3904, Q4 2N7002K, Q5 2N7002K, Q6 2N7002K

Commit message: Power done
Parts:
- added C? (x2): 0.1uF, Capacitor_SMD:C_0603_1608Metric, symbol Device:C_Small
- added C? (x5): 10uF, Capacitor_SMD:C_0603_1608Metric, symbol Device:C_Small
- added C? (x2): 2.2uF, Capacitor_SMD:C_0603_1608Metric, symbol Device:C_Small
- added C?: 1.0uF, Capacitor_SMD:C_0603_1608Metric, symbol Device:C_Small
- added C? (x4): 22pF, Capacitor_SMD:C_0603_1608Metric, symbol Device:C_Small
- added C?: 27pF, Capacitor_SMD:C_0603_1608Metric, symbol Device:C_Small
- added C?: 1uF, Capacitor_SMD:C_0603_1608Metric, symbol Device:C_Small
- added D?: D5V0L1B2LP-7B, Diode_SMD:D_01005_0402Metric, symbol Device:D_Zener
- added D? (x2): APTR3216-VFX, LED_SMD:LED_1206_3216Metric, symbol Device:LED
- added D?: BAT54A, Package_TO_SOT_SMD:SOT-23, symbol Diode:BAT54A
- added H? (x4): MountingHole_Pad, symbol Mechanical:MountingHole_Pad
- added JP?: Jumper, symbol Device:Jumper
- added L?: INDUCTOR, symbol pspice:INDUCTOR
- added Q? (x4): MBT3904DW1, Package_TO_SOT_SMD:SOT-363_SC-70-6, symbol Transistor_BJT:MBT3904DW1
- added R? (x2): 10kOhm, Resistor_SMD:R_0603_1608Metric, symbol Device:R_Small
- added R? (x3): 4.7kOhm, Resistor_SMD:R_0603_1608Metric, symbol Device:R_Small
- added R?: 148Ohm, Resistor_SMD:R_0603_1608Metric, symbol Device:R_Small
- added R?: 146Ohm, Resistor_SMD:R_0603_1608Metric, symbol Device:R_Small
- added R?: 10Ohm, Resistor_SMD:R_0603_1608Metric, symbol Device:R_Small
- added R?: 1Ohm, Resistor_SMD:R_0603_1608Metric, symbol Device:R_Small
- added R?: RQ5E035ATTCL, TRANS_RDR005N, symbol RQ5E035ATTCL:RQ5E035ATTCL
- added R? (x2): 40.2KOhm, Resistor_SMD:R_0603_1608Metric, symbol Device:R_Small
- added R?: 1kOhm, Resistor_SMD:R_0603_1608Metric, symbol Device:R_Small
- added R?: 0Ohm, Resistor_SMD:R_0603_1608Metric, symbol Device:R_Small
- added R?: 200kOhm, Resistor_SMD:R_0603_1608Metric, symbol Device:R_Small
- added R? (x2): 20kOhm, Resistor_SMD:R_0603_1608Metric, symbol Device:R_Small
- added SW?: SW_Push, symbol Switch:SW_Push
- added U?: APL5912KAC, Package_SO:HTSOP-8-1EP_3.9x4.9mm_P1.27mm_EP2.4x3.2mm, symbol APL5912KAC:APL5912KAC
Connections:
- net +5VSB: now also R?.2
- net +PS_3VSB: now also R?.2
- net +PS_5VSB: now also C?.1, D?.2 (A), R?.1
- net GND: now also C?.1, C?.1, C?.1, C?.1, C?.2, C?.2, C?.2, C?.2, C?.2, C?.2, C?.2, C?.2, C?.2, C?.2, C?.2, D?.2 (A), JP?.1, Q?.1 (E1), Q?.1 (E1), Q?.4 (E2), Q?.4 (E2), R?.1, R?.1, R?.2, R?.2, SW?.2, U?.1 (GND)
- net VCC: now also C?.1, D?.2 (A), R?.1, R?.2, R?.2
- net VCC3: now also L?.1, R?.1
- net SLP_S3_L: now reaches Q5.1 (G)
- net SLP_S3_L: now also D?.1
- new net: C?.2, R?.2, U?.2 (FB)
- new net: C?.2, R?.2, U?.6 (VCNTL)
- new net: R?.1, U?.7 (POK)
- new net: R?.1, U?.8 (EN)
- new net: D?.1 (K), R?.2 (x2)
- new net: H?.1, H?.1, H?.1, H?.1, R?.1
- new net: C?.1, R?.1, R?.2 (G)
- new net: Q?.2 (B1), R?.2
- new net: C?.2, D?.3, Q?.2 (B1), R?.2
- new net: Q?.5 (B2), Q?.6 (C1), R?.1
- new net +V1P0A_PWRGD: D?.2
- new net +V1P8S: R?.1
- new net +VDIMM: C?.1, C?.1, R?.3 (D), U?.5 (VIN), U?.9 (VIN)
- new net 1P5V_EN_B: Q?.5 (B2), Q?.6 (C1), R?.1
- new net 1P8V_EN: Q?.3 (C2), R?.1
- new net FP_PWRBTN: C?.1, D?.1 (K), JP?.2, R?.2, SW?.1
- new net SYS_PWRGD: Q?.3 (C2), R?.2
- new net V1P05S: C?.1, C?.1, C?.1, C?.1, C?.1, R?.1, R?.1, U?.3 (VOUT), U?.4 (VOUT)
- new net V1P0S_PG: R?.2
- new net V1P35S: C?.1, C?.2, R?.1, R?.1 (S)
- new net VCC3S: C?.2, L?.2
- new net VCORE_GFX_PG: R?.2

Commit message: Finished all except RAM and CPU
Parts:
- H1, H2, H3, H4: renamed from H?; footprint (none) -> MountingHole:MountingHole_3.2mm_M3_Pad
- JP1: renamed from JP?; footprint (none) -> Jumper:SolderJumper-2_P1.3mm_Open_RoundedPad1.0x1.5mm
- L16: renamed from L?; footprint (none) -> Inductor_SMD:L_0603_1608Metric
- R102, R103: footprint TRANS_RDR005N -> RQ5E035ATTCL:RQ5E035ATTCL
- R119: renamed from R?; footprint TRANS_RDR005N -> RQ5E035ATTCL:RQ5E035ATTCL
- R96, R98: footprint TRANS_RQ3C150 -> RQ3E180GNTB:RQ3E180GNTB
- SW1: renamed from SW?; footprint (none) -> Button_Switch_SMD:SW_SPST_TL3342
- gave numbers to parts that had none: 39
