File: PD4.sch (KiCad schematic (older format))
At the start: 33 parts

Commit message: Finished all except RAM and CPU
Parts:
- U30: renamed from U?; footprint DFN6_3X3P3 -> NCP606MN18T2G:NCP606MN18T2G
- gave numbers to parts that had none: 32
