File: PHASE.sch (KiCad schematic (older format))
At the start: 51 parts

Commit message: Finished all except RAM and CPU
Parts:
- C134, C135, C136: renamed from C?; footprint (none) -> Capacitor_Tantalum_SMD:CP_EIA-7343-20_Kemet-V
- L17, L18, L21, L22: renamed from L?; footprint (none) -> Inductor_SMD:L_0603_1608Metric
- L19, L20: renamed from L?; footprint IND_TDK_ACM2012_2P -> ACM2012-900-2P-T:ACM2012-900-2P-T
- U26, U27: renamed from U?; footprint (none) -> FDMS7602S:TRANS_FDMD8530
- gave numbers to parts that had none: 40
