File: SDCARD.sch (KiCad schematic (older format))
At the start: 17 parts

Commit message: finishing schematic
Parts:
- gave numbers to parts that had none: 17
Changed lines of the file:
@@
 $Descr A4 11693 8268
 encoding utf-8
-Sheet 7 20
+Sheet 7 21
 Title ""
 Date ""
@@
 $EndDescr
 $Comp
-L Connector:Micro_SD_Card J?
+L Connector:Micro_SD_Card J5
 U 1 1 5DAFBF76
 P 6100 3350
-F 0 "J?" H 6050 4067 50  0000 C CNN
+F 0 "J5" H 6050 4067 50  0000 C CNN
 F 1 "Micro_SD_Card" H 6050 3976 50  0000 C CNN
 F 2 "" H 7250 3650 50  0001 C CNN
@@
 $EndComp
 $Comp
-L Device:R_Small R?
+L Device:R_Small R75
 U 1 1 5DAFC66E
 P 3850 3750
-F 0 "R?" V 3654 3750 50  0000 C CNN
+F 0 "R75" V 3654 3750 50  0000 C CNN
 F 1 "33Ohm" V 3745 3750 50  0000 C CNN
 F 2 "Resistor_SMD:R_0603_1608Metric" H 3850 3750 50  0001 C CNN
@@
 	5200 3650 5050 3650
 $Comp
-L power:GND #PWR?
+L power:GND #PWR0172
 U 1 1 5DAFDA96
 P 5150 4150
-F 0 "#PWR?" H 5150 3900 50  0001 C CNN
+F 0 "#PWR0172" H 5150 3900 50  0001 C CNN
 F 1 "GND" H 5155 3977 50  0000 C CNN
 F 2 "" H 5150 4150 50  0001 C CNN
@@
 	5150 3550 5150 4100
 $Comp
-L Device:C_Small C?
+L Device:C_Small C65
 U 1 1 5DAFF73B
 P 6050 4100
-F 0 "C?" V 6150 4100 50  0000 C CNN
+F 0 "C65" V 6150 4100 50  0000 C CNN
 F 1 "8200pF" V 6250 4100 50  0000 C CNN
 F 2 "Resistor_SMD:R_0603_1608Metric" H 6050 4100 50  0001 C CNN
@@
 	5200 3050 4900 3050
 $Comp
-L power:+3V3 #PWR?
+L power:+3V3 #PWR0173
 U 1 1 5DB01C0A
 P 3950 1750
-F 0 "#PWR?" H 3950 1600 50  0001 C CNN
+F 0 "#PWR0173" H 3950 1600 50  0001 C CNN
 F 1 "+3V3" V 3965 1878 50  0000 L CNN
 F 2 "" H 3950 1750 50  0001 C CNN
@@
 $EndComp
 $Comp
-L Device:C_Small C?
+L Device:C_Small C63
 U 1 1 5DB01E84
 P 5700 2050
-F 0 "C?" H 5792 2096 50  0000 L CNN
+F 0 "C63" H 5792 2096 50  0000 L CNN
 F 1 "10uF" H 5792 2005 50  0000 L CNN
 F 2 "" H 5700 2050 50  0001 C CNN
@@
 $EndComp
 $Comp
-L Device:C_Small C?
+L Device:C_Small C64
 U 1 1 5DB01F86
 P 5950 2050
-F 0 "C?" H 6042 2096 50  0000 L CNN
+F 0 "C64" H 6042 2096 50  0000 L CNN
 F 1 "10uF" H 6042 2005 50  0000 L CNN
 F 2 "" H 5950 2050 50  0001 C CNN
@@
 	5700 1750 5950 1750
 $Comp
-L power:GND #PWR?
+L power:GND #PWR0174
 U 1 1 5DB02B78
 P 5700 2150
-F 0 "#PWR?" H 5700 1900 50  0001 C CNN
+F 0 "#PWR0174" H 5700 1900 50  0001 C CNN
 F 1 "GND" H 5705 1977 50  0000 C CNN
 F 2 "" H 5700 2150 50  0001 C CNN
@@
 $EndComp
 $Comp
-L power:GND #PWR?
+L power:GND #PWR0175
 U 1 1 5DB02BDC
 P 5950 2150
-F 0 "#PWR?" H 5950 1900 50  0001 C CNN
+F 0 "#PWR0175" H 5950 1900 50  0001 C CNN
 F 1 "GND" H 5955 1977 50  0000 C CNN
 F 2 "" H 5950 2150 50  0001 C CNN
@@
 	5000 1750 5700 1750
 $Comp
-L Device:R_Small R?
+L Device:R_Small R76
 U 1 1 5DB0336A
 P 4150 2000
-F 0 "R?" H 4209 2046 50  0000 L CNN
+F 0 "R76" H 4209 2046 50  0000 L CNN
 F 1 "100KOhm" H 4209 1955 50  0000 L CNN
 F 2 "Resistor_SMD:R_0603_1608Metric" H 4150 2000 50  0001 C CNN
@@
 $EndComp
 $Comp
-L Device:R_Small R?
+L Device:R_Small R77
 U 1 1 5DB04B47
 P 4250 2000
-F 0 "R?" H 4309 2046 50  0000 L CNN
+F 0 "R77" H 4309 2046 50  0000 L CNN
 F 1 "100KOhm" H 4309 1955 50  0000 L CNN
 F 2 "Resistor_SMD:R_0603_1608Metric" H 4250 2000 50  0001 C CNN
@@
 $EndComp
 $Comp
-L Device:R_Small R?
+L Device:R_Small R78
 U 1 1 5DB04D54
 P 4350 2000
-F 0 "R?" H 4409 2046 50  0000 L CNN
+F 0 "R78" H 4409 2046 50  0000 L CNN
 F 1 "100KOhm" H 4409 1955 50  0000 L CNN
 F 2 "Resistor_SMD:R_0603_1608Metric" H 4350 2000 50  0001 C CNN
@@
 $EndComp
 $Comp
-L Device:R_Small R?
+L Device:R_Small R79
 U 1 1 5DB04F11
 P 4450 2000
-F 0 "R?" H 4509 2046 50  0000 L CNN
+F 0 "R79" H 4509 2046 50  0000 L CNN
 F 1 "100KOhm" H 4509 1955 50  0000 L CNN
 F 2 "Resistor_SMD:R_0603_1608Metric" H 4450 2000 50  0001 C CNN
@@
 $EndComp
 $Comp
-L Device:R_Small R?
+L Device:R_Small R80
 U 1 1 5DB050AA
 P 4550 2000
-F 0 "R?" H 4609 2046 50  0000 L CNN
+F 0 "R80" H 4609 2046 50  0000 L CNN
 F 1 "100KOhm" H 4609 1955 50  0000 L CNN
 F 2 "Resistor_SMD:R_0603_1608Metric" H 4550 2000 50  0001 C CNN
@@
 $EndComp
 $Comp
-L Device:R_Small R?
+L Device:R_Small R81
 U 1 1 5DB051EF
 P 4650 2000
-F 0 "R?" H 4709 2046 50  0000 L CNN
+F 0 "R81" H 4709 2046 50  0000 L CNN
 F 1 "100KOhm" H 4709 1955 50  0000 L CNN
 F 2 "Resistor_SMD:R_0603_1608Metric" H 4650 2000 50  0001 C CNN
@@
 	4650 3750 4300 3750
 $Comp
-L Device:R_Small R?
+L Device:R_Small R74
 U 1 1 5DB0B5F6
 P 3850 3650
-F 0 "R?" V 3654 3650 50  0000 C CNN
+F 0 "R74" V 3654 3650 50  0000 C CNN
 F 1 "33Ohm" V 3745 3650 50  0000 C CNN
 F 2 "Resistor_SMD:R_0603_1608Metric" H 3850 3650 50  0001 C CNN
@@
 $EndComp
 $Comp
-L Device:R_Small R?
+L Device:R_Small R73
 U 1 1 5DB0B715
 P 3850 3450
-F 0 "R?" V 3654 3450 50  0000 C CNN
+F 0 "R73" V 3654 3450 50  0000 C CNN
 F 1 "33Ohm" V 3745 3450 50  0000 C CNN
 F 2 "Resistor_SMD:R_0603_1608Metric" H 3850 3450 50  0001 C CNN
@@
 $EndComp
 $Comp
-L Device:R_Small R?
+L Device:R_Small R72
 U 1 1 5DB0B8E6
 P 3850 3250
-F 0 "R?" V 3654 3250 50  0000 C CNN
+F 0 "R72" V 3654 3250 50  0000 C CNN
 F 1 "33Ohm" V 3745 3250 50  0000 C CNN
 F 2 "Resistor_SMD:R_0603_1608Metric" H 3850 3250 50  0001 C CNN
@@
 $EndComp
 $Comp
-L Device:R_Small R?
+L Device:R_Small R71
 U 1 1 5DB0BAEC
 P 3850 3150
-F 0 "R?" V 3654 3150 50  0000 C CNN
+F 0 "R71" V 3654 3150 50  0000 C CNN
 F 1 "33Ohm" V 3745 3150 50  0000 C CNN
 F 2 "Resistor_SMD:R_0603_1608Metric" H 3850 3150 50  0001 C CNN
@@
 $EndComp
 $Comp
-L Device:R_Small R?
+L Device:R_Small R70
 U 1 1 5DB0BBF7
 P 3850 3050
-F 0 "R?" V 3654 3050 50  0000 C CNN
+F 0 "R70" V 3654 3050 50  0000 C CNN
 F 1 "33Ohm" V 3745 3050 50  0000 C CNN
 F 2 "Resistor_SMD:R_0603_1608Metric" H 3850 3050 50  0001 C CNN
@@
 SD3_D1
 $Comp
-L TPD6E001RSER:TPD6E001RSER U?
+L TPD6E001RSER:TPD6E001RSER U8
 U 1 1 5DB0D39D
 P 4350 5750
-F 0 "U?" H 5450 6137 60  0000 C CNN
+F 0 "U8" H 5450 6137 60  0000 C CNN
 F 1 "TPD6E001RSER" H 5450 6031 60  0000 C CNN
 F 2 "TPD6E001RSER:TPD6E001RSER" H 5450 5990 60  0001 C CNN
@@
 	4700 3450 4450 3450
 $Comp
-L power:GND #PWR?
+L power:GND #PWR0176
 U 1 1 5DB18997
 P 4350 6150
-F 0 "#PWR?" H 4350 5900 50  0001 C CNN
+F 0 "#PWR0176" H 4350 5900 50  0001 C CNN
 F 1 "GND" H 4355 5977 50  0000 C CNN
 F 2 "" H 4350 6150 50  0001 C CNN
@@
 $EndComp
 $Comp
-L power:+3V3 #PWR?
+L power:+3V3 #PWR0177
 U 1 1 5DB18D6E
 P 6550 5750
-F 0 "#PWR?" H 6550 5600 50  0001 C CNN
+F 0 "#PWR0177" H 6550 5600 50  0001 C CNN
 F 1 "+3V3" H 6565 5923 50  0000 C CNN
 F 2 "" H 6550 5750 50  0001 C CNN

Commit message: Finished all except RAM and CPU
Parts:
- C63, C64: footprint (none) -> Capacitor_SMD:C_0603_1608Metric
- J5: footprint (none) -> Connector_Card:microSD_HC_Hirose_DM3AT-SF-PEJM5
Changed lines of the file:
@@
 $Descr A4 11693 8268
 encoding utf-8
-Sheet 7 23
+Sheet 7 24
 Title ""
 Date ""
@@
 F 0 "J5" H 6050 4067 50  0000 C CNN
 F 1 "Micro_SD_Card" H 6050 3976 50  0000 C CNN
-F 2 "" H 7250 3650 50  0001 C CNN
+F 2 "Connector_Card:microSD_HC_Hirose_DM3AT-SF-PEJM5" H 7250 3650 50  0001 C CNN
 F 3 "http://katalog.we-online.de/em/datasheet/693072010801.pdf" H 6100 3350 50  0001 C CNN
 	1    6100 3350
@@
 F 0 "C63" H 5792 2096 50  0000 L CNN
 F 1 "10uF" H 5792 2005 50  0000 L CNN
-F 2 "" H 5700 2050 50  0001 C CNN
+F 2 "Capacitor_SMD:C_0603_1608Metric" H 5700 2050 50  0001 C CNN
 F 3 "~" H 5700 2050 50  0001 C CNN
 	1    5700 2050
@@
 F 0 "C64" H 6042 2096 50  0000 L CNN
 F 1 "10uF" H 6042 2005 50  0000 L CNN
-F 2 "" H 5950 2050 50  0001 C CNN
+F 2 "Capacitor_SMD:C_0603_1608Metric" H 5950 2050 50  0001 C CNN
 F 3 "~" H 5950 2050 50  0001 C CNN
 	1    5950 2050
