File: USB.sch (KiCad schematic (older format))
At the start: 0 parts

Commit message: finishing schematic
Parts:
- added C52, C53, C54, C55, C56, C57, C58, C61, C62: 0.1uF, Capacitor_SMD:C_0603_1608Metric, symbol Device:C_Small
- added C59, C60: 22uF, Capacitor_SMD:C_0603_1608Metric, symbol Device:C_Small
- added F1: Fuse_Small, symbol Device:Fuse_Small
- added J2: USB_A, symbol Connector:USB_A
- added J3: USB3_A, symbol Connector:USB3_A
- added L10, L4: 0Ohm, Inductor_SMD:L_0603_1608Metric, symbol pspice:INDUCTOR
- added L3, L5, L6, L9: ACM2012-900, symbol Device:L_Coupled
- added L7, L8: 220Ohm, Inductor_SMD:L_0603_1608Metric, symbol pspice:INDUCTOR
- added U4, U7: TPD4S012DRYR, DRY6, symbol TPD4S012DRYR:TPD4S012DRYR
- added U5: TPS2066DR, D8, symbol TPS2066DR:TPS2066DR
- added U6: TPD4EUSB30, Package_SON:USON-10_2.5x1.0mm_P0.5mm, symbol Power_Protection:TPD4EUSB30
Connections:
- new net: J3.2 (D-), L9.4, U7.2 (D-)
- new net: J3.3 (D+), L9.2, U7.1 (D1+)
- new net: J3.5 (SSRX-), L6.4, U6.5 (D2-)
- new net: J3.6 (SSRX+), L6.2, U6.4 (D2+)
- new net: J3.8 (SSTX-), L5.4, U6.2 (D1-)
- new net: J3.9 (SSTX+), L5.2, U6.1 (D1+)
- new net: J2.2 (D-), L3.2, U4.1 (D1+)
- new net: J2.3 (D+), L3.4, U4.2 (D-)
- new net: C57.2, L5.1
- new net: C58.2, L5.3
- new net: L8.1, U5.6 (OUT2)
- new net: L7.1, U5.7 (OUT1)
- new net: C61.2, L10.2
- new net: C52.2, L4.2
- new net +5VSB: F1.1
- new net +USBVCC: C53.1, C54.1, C55.1, F1.2, U5.2 (IN)
- new net GND: C53.2, C54.2, C55.2, C56.2, C59.2, C60.2, C62.2, J2.4 (GND), J2.5 (Shield), J3.10 (SHIELD), J3.4 (GND), J3.7 (DRAIN), L10.1, L4.1, U4.4 (GND), U5.1 (GND), U6.3 (GND), U6.8 (GND), U7.4 (GND)
- new net USB3_RXN0: L6.3
- new net USB3_RXP0: L6.1
- new net USB3_TXN0: C58.1
- new net USB3_TXP0: C57.1
- new net USB_DN0: L9.3
- new net USB_DN1: L3.3
- new net USB_DP0: L9.1
- new net USB_DP1: L3.1
- new net USB_HOST_EN0: U5.3 (*EN1)
- new net USB_HOST_EN1: U5.4 (*EN2)
- new net USB_HOST_OC0: U5.8 (*OC1)
- new net USB_HOST_OC1: U5.5 (*OC2)
- new net VBUS1: C60.1, C61.1, C62.1, J3.1 (VBUS), L7.2, U7.6 (VBUS)
- new net VBUS2: C52.1, C56.1, C59.1, J2.1 (VBUS), L8.2, U4.6 (VBUS)

Commit message: finished fixes
Parts:
- added R? (x3): 10KOhm, Resistor_SMD:R_0603_1608Metric, symbol Device:R_Small
- added R? (x4): 2.2KOhm, Resistor_SMD:R_0603_1608Metric, symbol Device:R_Small
- added U?: TXS0104EYZTR, YZT12, symbol TXS0104EYZTR:TXS0104EYZTR
Connections:
- net +USBVCC: now also R?.1, R?.1, U?.B1 (VCCB)
- net GND: now also R?.2, R?.2, R?.2, R?.2, U?.D2
- net USB_HOST_EN0: now also R?.1, U?.A2
- net USB_HOST_EN1: now also R?.1, U?.D1
- net USB_HOST_OC0: now also R?.2, U?.A1
- net USB_HOST_OC1: now also R?.2, U?.A3
- new net: R?.2, U?.B3 (OE)
- new net +V1P8A: R?.1, U?.B2 (VCCA)
- new net SOC_USB_HOST_EN0: R?.1, U?.C2 (B2)
- new net SOC_USB_HOST_EN1: R?.1, U?.D3
- new net SOC_USB_HOST_OC0: U?.C1 (B1)
- new net SOC_USB_HOST_OC1: U?.C3 (B3)
Other:
- moved on the sheet: C53, C54, C55, C59, C60, F1, L7, L8, U5

Commit message: Finished all except RAM and CPU
Parts:
- F1: value Fuse_Small -> 2A; footprint (none) -> Fuse:Fuse_0603_1608Metric
- J2: footprint (none) -> Connector_USB:USB_A_CNCTech_1001-011-01101_Horizontal
- J3: footprint (none) -> Connector_USB:USB3_A_Molex_48393-001
- L3, L5, L6, L9: footprint (none) -> ACM2012-900-2P-T:ACM2012-900-2P-T
- U24: renamed from U?; footprint YZT12 -> TXS0104EYZTR:TXS0104EYZTR
- U4, U7: footprint DRY6 -> TPD4S012DRYR:TPD4S012DRYR
- U5: footprint D8 -> TPS2066DR:TPS2066DR
- gave numbers to parts that had none: 7
Changed lines of the file:
@@
 $Descr A4 11693 8268
 encoding utf-8
-Sheet 5 23
+Sheet 5 24
 Title ""
 Date ""
@@
 F 0 "J3" H 8170 4722 50  0000 R CNN
 F 1 "USB3_A" H 8170 4813 50  0000 R CNN
-F 2 "" H 8750 4950 50  0001 C CNN
+F 2 "Connector_USB:USB3_A_Molex_48393-001" H 8750 4950 50  0001 C CNN
 F 3 "~" H 8750 4950 50  0001 C CNN
 	1    8600 4850
@@
 F 0 "J2" H 1870 6097 50  0000 R CNN
 F 1 "USB_A" H 1870 6188 50  0000 R CNN
-F 2 "" H 2250 6150 50  0001 C CNN
+F 2 "Connector_USB:USB_A_CNCTech_1001-011-01101_Horizontal" H 2250 6150 50  0001 C CNN
 F 3 " ~" H 2250 6150 50  0001 C CNN
 	1    2100 6200
@@
 F 0 "U4" H 2850 4987 60  0000 C CNN
 F 1 "TPD4S012DRYR" H 2850 4881 60  0000 C CNN
-F 2 "DRY6" H 2850 4840 60  0001 C CNN
+F 2 "TPD4S012DRYR:TPD4S012DRYR" H 2850 4840 60  0001 C CNN
 F 3 "" H 1750 4600 60  0000 C CNN
 	1    1750 4600
@@
 F 0 "U7" H 9100 6137 60  0000 C CNN
 F 1 "TPD4S012DRYR" H 9100 6031 60  0000 C CNN
-F 2 "DRY6" H 9100 5990 60  0001 C CNN
+F 2 "TPD4S012DRYR:TPD4S012DRYR" H 9100 5990 60  0001 C CNN
 F 3 "" H 8000 5750 60  0000 C CNN
 	1    8000 5750
@@
 F 0 "L3" H 1300 6613 50  0000 C CNN
 F 1 "ACM2012-900" H 1300 6522 50  0000 C CNN
-F 2 "" H 1300 6150 50  0001 C CNN
+F 2 "ACM2012-900-2P-T:ACM2012-900-2P-T" H 1300 6150 50  0001 C CNN
 F 3 "~" H 1300 6150 50  0001 C CNN
 F 4 "90Ohm" H 1300 6431 50  0000 C CNN "Resistance"
@@
 F 0 "L9" H 7600 5463 50  0000 C CNN
 F 1 "ACM2012-900" H 7600 5372 50  0000 C CNN
-F 2 "" H 7600 5000 50  0001 C CNN
+F 2 "ACM2012-900-2P-T:ACM2012-900-2P-T" H 7600 5000 50  0001 C CNN
 F 3 "~" H 7600 5000 50  0001 C CNN
 F 4 "90Ohm" H 7600 5281 50  0000 C CNN "Resistance"
@@
 F 0 "L5" H 5000 5663 50  0000 C CNN
 F 1 "ACM2012-900" H 5000 5572 50  0000 C CNN
-F 2 "" H 5000 5200 50  0001 C CNN
+F 2 "ACM2012-900-2P-T:ACM2012-900-2P-T" H 5000 5200 50  0001 C CNN
 F 3 "~" H 5000 5200 50  0001 C CNN
 F 4 "90Ohm" H 5000 5481 50  0000 C CNN "Resistance"
@@
 F 0 "L6" H 6100 6663 50  0000 C CNN
 F 1 "ACM2012-900" H 6100 6572 50  0000 C CNN
-F 2 "" H 6100 6200 50  0001 C CNN
+F 2 "ACM2012-900-2P-T:ACM2012-900-2P-T" H 6100 6200 50  0001 C CNN
 F 3 "~" H 6100 6200 50  0001 C CNN
 F 4 "90Ohm" H 6100 6481 50  0000 C CNN "Resistance"
@@
 F 0 "U5" H 8300 2187 60  0000 C CNN
 F 1 "TPS2066DR" H 8300 2081 60  0000 C CNN
-F 2 "D8" H 8300 2040 60  0001 C CNN
+F 2 "TPS2066DR:TPS2066DR" H 8300 2040 60  0001 C CNN
 F 3 "" H 7100 1800 60  0000 C CNN
 	1    7100 1800
@@
 P 4850 1200
 F 0 "F1" H 4850 1385 50  0000 C CNN
-F 1 "Fuse_Small" H 4850 1294 50  0000 C CNN
-F 2 "" H 4850 1200 50  0001 C CNN
+F 1 "2A" H 4850 1294 50  0000 C CNN
+F 2 "Fuse:Fuse_0603_1608Metric" H 4850 1200 50  0001 C CNN
 F 3 "~" H 4850 1200 50  0001 C CNN
 	1    4850 1200
@@
 	2200 5800 2700 5800
 $Comp
-L TXS0104EYZTR:TXS0104EYZTR U?
+L TXS0104EYZTR:TXS0104EYZTR U24
 U 1 1 5DC65939
 P 1700 2300
-F 0 "U?" H 3000 2887 60  0000 C CNN
+F 0 "U24" H 3000 2887 60  0000 C CNN
 F 1 "TXS0104EYZTR" H 3000 2781 60  0000 C CNN
-F 2 "YZT12" H 3000 2840 60  0001 C CNN
+F 2 "TXS0104EYZTR:TXS0104EYZTR" H 3000 2840 60  0001 C CNN
 F 3 "" H 1700 2300 60  0000 C CNN
 	1    1700 2300
@@
 $EndComp
 $Comp
-L POWER:+V1P8A #PWR?
+L POWER:+V1P8A #PWR0227
 U 1 1 5DC669DD
 P 750 3300
-F 0 "#PWR?" H 750 3150 50  0001 C CNN
+F 0 "#PWR0227" H 750 3150 50  0001 C CNN
 F 1 "+V1P8A" V 768 3427 50  0000 L CNN
 F 2 "" H 750 3300 50  0001 C CNN
@@
 AR Path="/5DB78800/5DC7B3F0" Ref="R?"  Part="1"
 AR Path="/5DD54244/5DC7B3F0" Ref="R?"  Part="1"
-AR Path="/5DAC0636/5DC7B3F0" Ref="R?"  Part="1"
-F 0 "R?" H 1059 3346 50  0000 L CNN
+AR Path="/5DAC0636/5DC7B3F0" Ref="R106"  Part="1"
+F 0 "R106" H 1059 3346 50  0000 L CNN
 F 1 "10KOhm" H 1059 3255 50  0000 L CNN
 F 2 "Resistor_SMD:R_0603_1608Metric" H 1000 3300 50  0001 C CNN
@@
 	800  3300 750  3300
 $Comp
-L POWER:+USBVCC #PWR?
+L POWER:+USBVCC #PWR0228
 U 1 1 5DC84BB0
 P 850 1400
-F 0 "#PWR?" H 850 1250 50  0001 C CNN
+F 0 "#PWR0228" H 850 1250 50  0001 C CNN
 F 1 "+USBVCC" H 867 1573 50  0000 C CNN
 F 2 "" H 850 1400 50  0001 C CNN
@@
 AR Path="/5DB78800/5DC88BA9" Ref="R?"  Part="1"
 AR Path="/5DD54244/5DC88BA9" Ref="R?"  Part="1"
-AR Path="/5DAC0636/5DC88BA9" Ref="R?"  Part="1"
-F 0 "R?" H 1059 1496 50  0000 L CNN
+AR Path="/5DAC0636/5DC88BA9" Ref="R104"  Part="1"
+F 0 "R104" H 1059 1496 50  0000 L CNN
 F 1 "2.2KOhm" H 1059 1405 50  0000 L CNN
 F 2 "Resistor_SMD:R_0603_1608Metric" H 1000 1450 50  0001 C CNN
@@
 AR Path="/5DB78800/5DCEB5E6" Ref="R?"  Part="1"
 AR Path="/5DD54244/5DCEB5E6" Ref="R?"  Part="1"
-AR Path="/5DAC0636/5DCEB5E6" Ref="R?"  Part="1"
-F 0 "R?" H 1059 1746 50  0000 L CNN
+AR Path="/5DAC0636/5DCEB5E6" Ref="R105"  Part="1"
+F 0 "R105" H 1059 1746 50  0000 L CNN
 F 1 "2.2KOhm" H 1059 1655 50  0000 L CNN
 F 2 "Resistor_SMD:R_0603_1608Metric" H 1000 1700 50  0001 C CNN
@@
 AR Path="/5DB78800/5DCFDA40" Ref="R?"  Part="1"
 AR Path="/5DD54244/5DCFDA40" Ref="R?"  Part="1"
-AR Path="/5DAC0636/5DCFDA40" Ref="R?"  Part="1"
-F 0 "R?" H 2209 1396 50  0000 L CNN
+AR Path="/5DAC0636/5DCFDA40" Ref="R107"  Part="1"
+F 0 "R107" H 2209 1396 50  0000 L CNN
 F 1 "10KOhm" H 2209 1305 50  0000 L CNN
 F 2 "Resistor_SMD:R_0603_1608Metric" H 2150 1350 50  0001 C CNN
@@
 AR Path="/5DB78800/5DCFDD46" Ref="R?"  Part="1"
 AR Path="/5DD54244/5DCFDD46" Ref="R?"  Part="1"
-AR Path="/5DAC0636/5DCFDD46" Ref="R?"  Part="1"
-F 0 "R?" H 2209 1546 50  0000 L CNN
+AR Path="/5DAC0636/5DCFDD46" Ref="R108"  Part="1"
+F 0 "R108" H 2209 1546 50  0000 L CNN
 F 1 "10KOhm" H 2209 1455 50  0000 L CNN
 F 2 "Resistor_SMD:R_0603_1608Metric" H 2150 1500 50  0001 C CNN
@@
 $EndComp
 $Comp
-L power:GND #PWR?
+L power:GND #PWR0229
 U 1 1 5DD031AA
 P 2450 1650
-F 0 "#PWR?" H 2450 1400 50  0001 C CNN
+F 0 "#PWR0229" H 2450 1400 50  0001 C CNN
 F 1 "GND" H 2455 1477 50  0000 C CNN
 F 2 "" H 2450 1650 50  0001 C CNN
@@
 AR Path="/5DB78800/5DD41CD6" Ref="R?"  Part="1"
 AR Path="/5DD54244/5DD41CD6" Ref="R?"  Part="1"
-AR Path="/5DAC0636/5DD41CD6" Ref="R?"  Part="1"
-F 0 "R?" H 4559 3846 50  0000 L CNN
+AR Path="/5DAC0636/5DD41CD6" Ref="R109"  Part="1"
+F 0 "R109" H 4559 3846 50  0000 L CNN
 F 1 "2.2KOhm" H 4559 3755 50  0000 L CNN
 F 2 "Resistor_SMD:R_0603_1608Metric" H 4500 3800 50  0001 C CNN
@@
 AR Path="/5DB78800/5DD42536" Ref="R?"  Part="1"
 AR Path="/5DD54244/5DD42536" Ref="R?"  Part="1"
-AR Path="/5DAC0636/5DD42536" Ref="R?"  Part="1"
-F 0 "R?" H 4859 3846 50  0000 L CNN
+AR Path="/5DAC0636/5DD42536" Ref="R110"  Part="1"
+F 0 "R110" H 4859 3846 50  0000 L CNN
 F 1 "2.2KOhm" H 4859 3755 50  0000 L CNN
 F 2 "Resistor_SMD:R_0603_1608Metric" H 4800 3800 50  0001 C CNN
@@
 	4800 2300 4300 2300
 $Comp
-L power:GND #PWR?
+L power:GND #PWR0230
 U 1 1 5DD5EAEB
 P 4800 4100
-F 0 "#PWR?" H 4800 3850 50  0001 C CNN
+F 0 "#PWR0230" H 4800 3850 50  0001 C CNN
 F 1 "GND" H 4805 3927 50  0000 C CNN
 F 2 "" H 4800 4100 50  0001 C CNN
@@
 Connection ~ 4800 3900
 $Comp
-L power:GND #PWR?
+L power:GND #PWR0231
 U 1 1 5DD6EF79
 P 4550 2600
-F 0 "#PWR?" H 4550 2350 50  0001 C CNN
+F 0 "#PWR0231" H 4550 2350 50  0001 C CNN
 F 1 "GND" H 4555 2427 50  0000 C CNN
 F 2 "" H 4550 2600 50  0001 C CNN
