File: CPU_A.sch (KiCad schematic (older format))
At the start: 1 part

Commit message: finishing schematic
Parts:
- gave numbers to parts that had none: 1
Changed lines of the file:
@@
 $Descr A4 11693 8268
 encoding utf-8
-Sheet 8 20
+Sheet 8 21
 Title ""
 Date ""
@@
 $EndDescr
 $Comp
-L atom:atom_A U?
+L atom:atom_A U9
 U 1 1 5DB66C32
 P 3150 400
-F 0 "U?" H 4400 690 60  0000 C CNN
+F 0 "U9" H 4400 690 60  0000 C CNN
 F 1 "atom_A" H 4400 584 60  0000 C CNN
 F 2 "" H 3350 450 60  0001 L CNN

Commit message: Finished all except RAM and CPU
Parts:
- added C? (x2): 18pF, Capacitor_SMD:C_0603_1608Metric, symbol Device:C_Small
- added R?: 10MOhm, Resistor_SMD:R_0603_1608Metric, symbol Device:R_Small
- added Y?: Crystal, Crystal:Crystal_SMD_3215-2Pin_3.2x1.5mm, symbol Device:Crystal
Connections:
- net at U9.A9 (ILB_RTC_X2): now also C?.2, R?.1, Y?.1
- net at U9.C9 (ILB_RTC_X1): now also C?.2, R?.2, Y?.2
- new net GND: C?.1, C?.1
Changed lines of the file:
@@
 $Descr A4 11693 8268
 encoding utf-8
-Sheet 8 23
+Sheet 8 24
 Title ""
 Date ""
@@
 	1    0    0    -1
 $EndComp
+$Comp
+L Device:Crystal Y?
+U 1 1 5DD612D9
+P 10200 1200
+F 0 "Y?" H 10200 1468 50  0000 C CNN
+F 1 "Crystal" H 10200 1377 50  0000 C CNN
+F 2 "Crystal:Crystal_SMD_3215-2Pin_3.2x1.5mm" H 10200 1200 50  0001 C CNN
+F 3 "~" H 10200 1200 50  0001 C CNN
+	1    10200 1200
+	1    0    0    -1
+$EndComp
+$Comp
+L Device:R_Small R?
+U 1 1 5DD693DC
+P 10200 850
+AR Path="/5DB78800/5DD693DC" Ref="R?"  Part="1"
+AR Path="/5DB66240/5DD693DC" Ref="R?"  Part="1"
+F 0 "R?" H 10259 896 50  0000 L CNN
+F 1 "10MOhm" H 10259 805 50  0000 L CNN
+F 2 "Resistor_SMD:R_0603_1608Metric" H 10200 850 50  0001 C CNN
+F 3 "~" H 10200 850 50  0001 C CNN
+	1    10200 850
+	0    -1   -1   0
+$EndComp
+$Comp
+L Device:C_Small C?
+U 1 1 5DD693E2
+P 9900 1450
+AR Path="/5DB78800/5DD693E2" Ref="C?"  Part="1"
+AR Path="/5DB66240/5DD693E2" Ref="C?"  Part="1"
+F 0 "C?" H 9992 1496 50  0000 L CNN
+F 1 "18pF" H 9992 1405 50  0000 L CNN
+F 2 "Capacitor_SMD:C_0603_1608Metric" H 9900 1450 50  0001 C CNN
+F 3 "~" H 9900 1450 50  0001 C CNN
+	1    9900 1450
+	-1   0    0    1
+$EndComp
+Wire Wire Line
+	10100 850  9900 850
+Wire Wire Line
+	9900 850  9900 1200
+Wire Wire Line
+	9900 1200 10050 1200
+Wire Wire Line
+	9900 1200 9900 1350
+Connection ~ 9900 1200
+$Comp
+L Device:C_Small C?
+U 1 1 5DD6B8D6
+P 10500 1450
+AR Path="/5DB78800/5DD6B8D6" Ref="C?"  Part="1"
+AR Path="/5DB66240/5DD6B8D6" Ref="C?"  Part="1"
+F 0 "C?" H 10592 1496 50  0000 L CNN
+F 1 "18pF" H 10592 1405 50  0000 L CNN
+F 2 "Capacitor_SMD:C_0603_1608Metric" H 10500 1450 50  0001 C CNN
+F 3 "~" H 10500 1450 50  0001 C CNN
+	1    10500 1450
+	-1   0    0    1
+$EndComp
+Wire Wire Line
+	9900 1550 9900 1600
+Wire Wire Line
+	10500 1600 10500 1550
+$Comp
+L power:GND #PWR?
+U 1 1 5DD6C515
+P 10200 1750
+F 0 "#PWR?" H 10200 1500 50  0001 C CNN
+F 1 "GND" H 10205 1577 50  0000 C CNN
+F 2 "" H 10200 1750 50  0001 C CNN
+F 3 "" H 10200 1750 50  0001 C CNN
+	1    10200 1750
+	1    0    0    -1
+$EndComp
+Wire Wire Line
+	10200 1750 10200 1600
+Wire Wire Line
+	10500 850  10500 1200
+Wire Wire Line
+	10300 850  10500 850
+Wire Wire Line
+	10350 1200 10500 1200
+Connection ~ 10500 1200
+Wire Wire Line
+	10500 1200 10500 1350
+Wire Wire Line
+	9900 1600 10200 1600
+Connection ~ 10200 1600
+Wire Wire Line
+	10200 1600 10500 1600
+Wire Wire Line
+	9250 1400 5650 1400
+Wire Wire Line
+	9250 650  10500 650
+Wire Wire Line
+	10500 650  10500 850
+Wire Wire Line
+	9250 650  9250 1400
+Connection ~ 10500 850
+Wire Wire Line
+	5650 7900 6900 7900
+Wire Wire Line
+	6900 7900 6900 6250
+Wire Wire Line
+	6900 6250 9550 6250
+Wire Wire Line
+	9550 6250 9550 850
+Wire Wire Line
+	9550 850  9900 850
+Connection ~ 9900 850
 $EndSCHEMATC

Commit message: first gbrs
Parts:
- added C171, C173: 27pF, Capacitor_SMD:C_0603_1608Metric, symbol Device:C_Small
- added C172: 10pF, Capacitor_SMD:C_0603_1608Metric, symbol Device:C_Small
- added JP2: Jumper, Jumper:SolderJumper-2_P1.3mm_Open_RoundedPad1.0x1.5mm, symbol Device:Jumper
- added R159, R161, R163, R164, R165: 10KOhm, Resistor_SMD:R_0603_1608Metric, symbol Device:R_Small
- added R160: 402Ohm, Resistor_SMD:R_0603_1608Metric, symbol Device:R_Small
- added R162: 1KOhm, Resistor_SMD:R_0603_1608Metric, symbol Device:R_Small
- added R166, R187, R188, R189, R190: 0Ohm, Resistor_SMD:R_0603_1608Metric, symbol Device:R_Small
- added R167: 73.2Ohm, Resistor_SMD:R_0603_1608Metric, symbol Device:R_Small
- added R168, R169, R172: 49.9Ohm, Resistor_SMD:R_0603_1608Metric, symbol Device:R_Small
- added R170, R171: 150Ohm, Resistor_SMD:R_0603_1608Metric, symbol Device:R_Small
- added R173: 357Ohm, Resistor_SMD:R_0603_1608Metric, symbol Device:R_Small
- added R185: 4.02KOhm, Resistor_SMD:R_0603_1608Metric, symbol Device:R_Small
- added R186: 47.5Ohm, Resistor_SMD:R_0603_1608Metric, symbol Device:R_Small
- added R191: 1MOhm, Resistor_SMD:R_0603_1608Metric, symbol Device:R_Small
- added TP1, TP2: TestPoint, TestPoint:TestPoint_Pad_D2.0mm, symbol Connector:TestPoint
- added Y2: Crystal_GND24_Small, Crystal:Crystal_SMD_3225-4Pin_3.2x2.5mm_HandSoldering, symbol Device:Crystal_GND24_Small
- U9: value atom_A -> atom_A_copy; footprint (none) -> Atom:FCBGA11702; symbol atom:atom_A -> atom:atom_A_copy
- gave numbers to parts that had none: 4
Connections:
- net GND: now also U9.AY3 (VGA_IRTN), C171.2, C172.1, C173.1, R160.1, R164.2, R165.2, R168.2, R169.1, R170.1, R171.1, R172.1, R173.1, R185.1, R186.2
- net at U9.A21 (PCU_SPI_MOSI): now also R187.1
- net at U9.AD13 (ICLK_RCOMP): now also R186.1
- net at U9.AD14 (ICLK_ICOMP): now also R185.2
- net at U9.AH10 (ICLK_OSCOUT): now also C173.2, R191.2, Y2.3
- net at U9.AH12 (ICLK_OSCIN): now also C171.1, R191.1, Y2.1
- net SD3_D0: now reaches U9.AT28 (SD3_D[0])
- net SD3_D2: now reaches U9.AU28 (SD3_D[2])
- net SD3_CMD: now reaches U9.AV28 (SD3_CMD)
- net at U9.AW1 (VGA_IREF): now also R173.2
- net at U9.AY18 (MMC1_RCOMP): now also R172.2
- net SD3_CLK: now reaches U9.AY26 (SD3_CLK)
- net at U9.B22 (PCU_SPI_MISO): now also R188.2
- net SD3_D3: now reaches U9.BA26 (SD3_D[3])
- net LPE_I2SFRM: now reaches U9.BA30 (LPE_I2S2_FRM)
- net at U9.BC1 (VGA_DDCCLK): now also R171.2
- net at U9.BC2 (VGA_DDCDATA): now also R170.2
- net SD3_CD#: now reaches U9.BC24 (SD3_CD#)
- net SD3_CD#: now also R166.1
- net LPE_I2S_DATOUT: now reaches U9.BC30 (LPE_I2S2_DATAOUT)
- net at U9.BD22 (SD3_PWREN#): now also TP1.1
- net SD3_D1: now reaches U9.BD26 (SD3_D[1])
- net LPE_I2S_DATIN: now reaches U9.BD28 (LPE_I2S2_DATAIN)
- net at U9.BD5 (SD3_WP): now also JP2.2, R160.2
- net at U9.BF20 (HDA_LPE_RCOMP): now also R169.2
- net at U9.BF22 (SD3_1P8EN): now also TP2.1
- net at U9.BF26 (SD3_RCOMP): now also R168.1
- net LPE_I2S_CLK: now reaches U9.BF28 (LPE_I2S2_CLK)
- net at U9.C22 (PCU_SPI_CLK): now also R190.1
- net at U9.C23 (PCU_SPI_CS[0]#): now also R189.1
- net VR_HOT_L: now reaches U9.C24 (PROCHOT#)
- net VR_HOT_L: now also R167.1
- new net: JP2.1, R159.1
- new net: R162.2, R165.1
- new net +V1P8S: R159.2, R161.2, R163.2
- new net GPIO_S5_10_UNLOCK: R162.1
- new net GPIO_s0_SC_56: R163.1, R164.1
- new net LPE_I2S_FRM: R161.1
- new net SD3_WP: R166.2
- new net SOC_SPI_CLK-R: C172.2, R190.2
- new net SOC_SPI_CSOB-R: R189.2
- new net SOC_SPI_MISO-R: R188.1
- new net SOC_SPI_MOSI-R: R187.2
- new net V1P0S: R167.2
