File: CPU_B.sch (KiCad schematic (older format))
At the start: 1 part

Commit message: finishing schematic
Parts:
- gave numbers to parts that had none: 1
Changed lines of the file:
@@
 $Descr A4 11693 8268
 encoding utf-8
-Sheet 9 20
+Sheet 9 21
 Title ""
 Date ""
@@
 $EndDescr
 $Comp
-L atom:atom_B U?
+L atom:atom_B U10
 U 1 1 5DB6DF60
 P 5200 -300
-F 0 "U?" H 5700 -10 60  0000 C CNN
+F 0 "U10" H 5700 -10 60  0000 C CNN
 F 1 "atom_B" H 5700 -116 60  0000 C CNN
 F 2 "" H 5400 -250 60  0001 L CNN

Commit message: first gbrs
Parts:
- U10: value atom_B -> atom_A_copy; footprint (none) -> Atom:FCBGA11702; symbol atom:atom_B -> atom:atom_A_copy
Connections:
- net GND: now reaches U10.A11 (VSS)
- net GND: now also U10.A15 (VSS), U10.A19 (VSS), U10.A23 (VSS), U10.A27 (VSS), U10.A3 (VSS), U10.A31 (VSS), U10.A35 (VSS), U10.A39 (VSS), U10.A43 (VSS), U10.A47 (VSS), U10.A49 (VSS), U10.A5 (VSS), U10.A51 (VSS), U10.A52 (VSS), U10.A6 (VSS), U10.AA1 (VSS), U10.AA16 (VSS), U10.AA19 (VSS), U10.AA21 (VSS), U10.AA3 (VSS), U10.AA32 (VSS), U10.AA35 (VSS), U10.AA38 (VSS), U10.AA53 (VSS), U10.AB10 (VSS), U10.AB4 (VSS), U10.AB41 (VSS), U10.AB45 (VSS), U10.AB47 (VSS), U10.AB48 (VSS), U10.AB50 (VSS), U10.AB51 (VSS), U10.AB6 (VSS), U10.AC16 (VSS), U10.AC18 (VSS), U10.AC19 (VSS), U10.AC21 (VSS), U10.AC25 (VSS), U10.AC33 (VSS), U10.AC35 (VSS), U10.AC36 (VSS), U10.AC38 (VSS), U10.AD19 (VSS), U10.AD21 (VSS), U10.AD25 (VSS), U10.AD32 (VSS), U10.AD33 (VSS), U10.AD47 (VSS), U10.AD7 (VSS), U10.AE1 (VSS), U10.AE11 (VSS), U10.AE12 (VSS), U10.AE14 (VSS), U10.AE3 (VSS), U10.AE4 (VSS), U10.AE40 (VSS), U10.AE42 (VSS), U10.AE43 (VSS), U10.AE45 (VSS), U10.AE46 (VSS), U10.AE6 (VSS), U10.AE8 (VSS), U10.AE9 (VSS), U10.B2 (VSS), U10.B52 (VSS), U10.B53 (VSS), U10.C1 (VSS), U10.C14 (VSS), U10.C31 (VSS), U10.C34 (VSS), U10.C39 (VSS), U10.C42 (VSS), U10.C45 (VSS), U10.C49 (VSS), U10.C53 (VSS), U10.D12 (VSS), U10.D16 (VSS), U10.D24 (VSS), U10.D30 (VSS), U10.D36 (VSS), U10.D38 (VSS), U10.E1 (VSS), U10.E19 (VSS), U10.E35 (VSS), U10.E53 (VSS), U10.E8 (VSS), U10.F19 (VSS), U10.F2 (VSS), U10.F24 (VSS), U10.F27 (VSS), U10.F30 (VSS), U10.F35 (VSS), U10.F5 (VSS), U10.F7 (VSS), U10.G10 (VSS), U10.G20 (VSS), U10.G22 (VSS), U10.G26 (VSS), U10.G28 (VSS), U10.G32 (VSS), U10.G34 (VSS), U10.G42 (VSS), U10.J35 (VSS), U10.J40 (VSS), U10.J53 (VSS), U10.K14 (VSS), U10.K22 (VSS), U10.K32 (VSS), U10.K36 (VSS), U10.K4 (VSS), U10.K50 (VSS), U10.K9 (VSS), U10.L13 (VSS), U10.L19 (VSS), U10.L27 (VSS), U10.L35 (VSS), U10.M19 (VSS), U10.M26 (VSS), U10.M27 (VSS), U10.M28 (VSS), U10.M34 (VSS), U10.M35 (VSS), U10.M38 (VSS), U10.M47 (VSS), U10.M51 (VSS), U10.N1 (VSS), U10.N16 (VSS), U10.N38 (VSS), U10.N51 (VSS), U10.P13 (VSS), U10.P16 (VSS), U10.P19 (VSS), U10.P20 (VSS), U10.P24 (VSS), U10.P32 (VSS), U10.P35 (VSS), U10.P38 (VSS), U10.P4 (VSS), U10.P47 (VSS), U10.P52 (VSS), U10.P9 (VSS), U10.T40 (VSS), U10.U1 (VSS), U10.U11 (VSS), U10.U12 (VSS), U10.U14 (VSS), U10.U21 (VSS), U10.U3 (VSS), U10.U30 (VSS), U10.U32 (VSS), U10.U40 (VSS), U10.U42 (VSS), U10.U43 (VSS), U10.U45 (VSS), U10.U46 (VSS), U10.U48 (VSS), U10.U49 (VSS), U10.U5 (VSS), U10.U51 (VSS), U10.U53 (VSS), U10.U6 (VSS), U10.U8 (VSS), U10.U9 (VSS), U10.V12 (VSS), U10.V16 (VSS), U10.V19 (VSS), U10.V21 (VSS), U10.V35 (VSS), U10.V40 (VSS), U10.V44 (VSS), U10.V51 (VSS), U10.V7 (VSS), U10.Y10 (VSS), U10.Y14 (VSS), U10.Y16 (VSS), U10.Y21 (VSS), U10.Y25 (VSS), U10.Y33 (VSS), U10.Y41 (VSS), U10.Y44 (VSS), U10.Y7 (VSS), U10.Y9 (VSS)
