File: CPU_C.sch (KiCad schematic (older format))
At the start: 1 part

Commit message: finishing schematic
Parts:
- gave numbers to parts that had none: 1
Changed lines of the file:
@@
 $Descr A4 11693 8268
 encoding utf-8
-Sheet 10 20
+Sheet 10 21
 Title ""
 Date ""
@@
 $EndDescr
 $Comp
-L atom:atom_C U?
+L atom:atom_C U11
 U 1 1 5DB723E3
 P 5150 -350
-F 0 "U?" H 5650 -60 60  0000 C CNN
+F 0 "U11" H 5650 -60 60  0000 C CNN
 F 1 "atom_C" H 5650 -166 60  0000 C CNN
 F 2 "" H 5350 -300 60  0001 L CNN

Commit message: first gbrs
Parts:
- U11: value atom_C -> atom_A_copy; footprint (none) -> Atom:FCBGA11702; symbol atom:atom_C -> atom:atom_A_copy
Connections:
- net GND: now reaches U11.AE48 (VSS)
- net GND: now also U11.AE50 (VSS), U11.AE51 (VSS), U11.AE53 (VSS), U11.AF10 (VSS), U11.AF12 (VSS), U11.AF25 (VSS), U11.AF32 (VSS), U11.AF47 (VSS), U11.AG16 (VSS), U11.AG25 (VSS), U11.AG36 (VSS), U11.AG38 (VSS), U11.AH4 (VSS), U11.AH41 (VSS), U11.AH45 (VSS), U11.AH47 (VSS), U11.AH48 (VSS), U11.AH50 (VSS), U11.AH51 (VSS), U11.AH6 (VSS), U11.AH7 (VSS), U11.AH9 (VSS), U11.AJ1 (VSS), U11.AJ16 (VSS), U11.AJ21 (VSS), U11.AJ25 (VSS), U11.AJ27 (VSS), U11.AJ29 (VSS), U11.AJ3 (VSS), U11.AJ30 (VSS), U11.AJ32 (VSS), U11.AJ33 (VSS), U11.AJ35 (VSS), U11.AJ38 (VSS), U11.AJ53 (VSS), U11.AK10 (VSS), U11.AK14 (VSS), U11.AK16 (VSS), U11.AK33 (VSS), U11.AK41 (VSS), U11.AK44 (VSS), U11.AM12 (VSS), U11.AM19 (VSS), U11.AM24 (VSS), U11.AM25 (VSS), U11.AM29 (VSS), U11.AM33 (VSS), U11.AM35 (VSS), U11.AM36 (VSS), U11.AM40 (VSS), U11.AM44 (VSS), U11.AM51 (VSS), U11.AM7 (VSS), U11.AN1 (VSS), U11.AN11 (VSS), U11.AN12 (VSS), U11.AN14 (VSS), U11.AN16 (VSSA), U11.AN22 (VSS), U11.AN3 (VSS), U11.AN33 (VSS), U11.AN35 (VSS), U11.AN36 (VSS), U11.AN38 (VSS), U11.AN40 (VSS), U11.AN42 (VSS), U11.AN43 (VSS), U11.AN45 (VSS), U11.AN46 (VSS), U11.AN48 (VSS), U11.AN49 (VSS), U11.AN5 (VSS), U11.AN51 (VSS), U11.AN53 (VSS), U11.AN6 (VSS), U11.AN8 (VSS), U11.AN9 (VSS), U11.AP40 (VSS), U11.AT12 (VSS), U11.AT16 (VSS), U11.AT19 (VSS), U11.AT24 (VSS), U11.AT27 (VSS), U11.AT30 (VSS), U11.AT35 (VSS), U11.AT38 (VSS), U11.AT4 (VSS), U11.AT47 (VSS), U11.AT52 (VSS), U11.AU1 (VSS), U11.AU24 (VSS), U11.AU3 (VSS), U11.AU30 (VSS), U11.AU38 (VSS), U11.AU51 (VSS), U11.AV12 (VSS), U11.AV13 (VSS), U11.AV14 (VSS), U11.AV18 (VSS), U11.AV19 (VSS), U11.AV24 (VSS), U11.AV27 (VSS), U11.AV30 (VSS), U11.AV35 (VSS), U11.AV38 (VSS), U11.AV47 (VSS), U11.AV51 (VSS), U11.AV7 (VSS), U11.AW13 (VSS), U11.AW19 (VSS), U11.AW27 (VSS), U11.AW3 (VSS), U11.AW35 (VSS), U11.AY10 (VSS), U11.AY22 (VSS), U11.AY32 (VSS), U11.AY36 (VSS), U11.AY4 (VSS), U11.AY50 (VSS), U11.AY9 (VSS), U11.BA14 (VSS), U11.BA19 (VSS), U11.BA22 (VSS), U11.BA27 (VSS), U11.BA32 (VSS), U11.BA35 (VSS), U11.BA40 (VSS), U11.BA53 (VSS), U11.BB19 (VSS), U11.BB27 (VSS), U11.BB35 (VSS), U11.BC20 (VSS), U11.BC22 (VSS), U11.BC26 (VSS), U11.BC28 (VSS), U11.BC32 (VSS), U11.BC34 (VSS), U11.BC42 (VSS), U11.BD19 (VSS), U11.BD24 (VSS), U11.BD27 (VSS), U11.BD30 (VSS), U11.BD35 (VSS), U11.BE1 (VSS), U11.BE19 (VSS), U11.BE2 (VSS), U11.BE35 (VSS), U11.BE53 (VSS), U11.BE8 (VSS), U11.BF12 (VSS), U11.BF16 (VSS), U11.BF24 (VSS), U11.BF30 (VSS), U11.BF36 (VSS), U11.BF38 (VSS), U11.BF4 (VSS), U11.BG1 (VSS), U11.BG31 (VSS), U11.BG34 (VSS), U11.BG39 (VSS), U11.BG42 (VSS), U11.BG45 (VSS), U11.BG49 (VSS), U11.BG53 (VSS), U11.BH1 (VSS), U11.BH2 (VSS), U11.BH52 (VSS), U11.BH53 (VSS), U11.BJ11 (VSS), U11.BJ15 (VSS), U11.BJ19 (VSS), U11.BJ2 (VSS), U11.BJ23 (VSS), U11.BJ27 (VSS), U11.BJ3 (VSS), U11.BJ31 (VSS), U11.BJ35 (VSS), U11.BJ39 (VSS), U11.BJ43 (VSS), U11.BJ47 (VSS), U11.BJ49 (VSS), U11.BJ5 (VSS), U11.BJ51 (VSS), U11.BJ52 (VSS), U11.BJ7 (VSS)
