File: CPU_E.sch (KiCad schematic (older format))
At the start: 1 part

Commit message: finishing schematic
Parts:
- gave numbers to parts that had none: 1
Changed lines of the file:
@@
 $Descr A4 11693 8268
 encoding utf-8
-Sheet 12 20
+Sheet 12 21
 Title ""
 Date ""
@@
 $EndDescr
 $Comp
-L atom:atom_E U?
+L atom:atom_E U13
 U 1 1 5DB7B823
 P 4250 2350
-F 0 "U?" H 6050 -1647 60  0000 C CNN
+F 0 "U13" H 6050 -1647 60  0000 C CNN
 F 1 "atom_E" H 6050 -1753 60  0000 C CNN
 F 2 "" H 4400 2400 60  0001 R CNN

Commit message: first gbrs
Parts:
- U13: value atom_E -> atom_A_copy; footprint (none) -> Atom:FCBGA11702; symbol atom:atom_E -> atom:atom_A_copy
Changed lines of the file:
@@
 $EndDescr
 $Comp
-L atom:atom_E U13
-U 1 1 5DB7B823
+L atom:atom_A_copy U13
+U 5 1 5DB7B823
 P 4250 2350
 F 0 "U13" H 6050 -1647 60  0000 C CNN
-F 1 "atom_E" H 6050 -1753 60  0000 C CNN
-F 2 "" H 4400 2400 60  0001 R CNN
+F 1 "atom_A_copy" H 6050 -1753 60  0000 C CNN
+F 2 "Atom:FCBGA11702" H 4400 2400 60  0001 R CNN
 F 3 "" H 4400 2200 60  0001 R CNN
-	1    4250 2350
+	5    4250 2350
 	1    0    0    -1
 $EndComp
