File: CPU_F.sch (KiCad schematic (older format))
At the start: 1 part

Commit message: finishing schematic
Parts:
- gave numbers to parts that had none: 1
Changed lines of the file:
@@
 $Descr A4 11693 8268
 encoding utf-8
-Sheet 13 20
+Sheet 13 21
 Title ""
 Date ""
@@
 $EndDescr
 $Comp
-L atom:atom_F U?
+L atom:atom_F U14
 U 1 1 5DB7D1E2
 P 1750 -2750
-F 0 "U?" H 4000 -1247 60  0000 C CNN
+F 0 "U14" H 4000 -1247 60  0000 C CNN
 F 1 "atom_F" H 4000 -1353 60  0000 C CNN
 F 2 "" H 1900 -2700 60  0001 R CNN

Commit message: first gbrs
Parts:
- U14: value atom_F -> atom_A_copy; footprint (none) -> Atom:FCBGA11702; symbol atom:atom_F -> atom:atom_A_copy
Changed lines of the file:
@@
 $EndDescr
 $Comp
-L atom:atom_F U14
-U 1 1 5DB7D1E2
+L atom:atom_A_copy U14
+U 6 1 5DB7D1E2
 P 1750 -2750
 F 0 "U14" H 4000 -1247 60  0000 C CNN
-F 1 "atom_F" H 4000 -1353 60  0000 C CNN
-F 2 "" H 1900 -2700 60  0001 R CNN
+F 1 "atom_A_copy" H 4000 -1353 60  0000 C CNN
+F 2 "Atom:FCBGA11702" H 1900 -2700 60  0001 R CNN
 F 3 "" H 1900 -2900 60  0001 R CNN
-	1    1750 -2750
+	6    1750 -2750
 	1    0    0    -1
 $EndComp
