File: CPU_G.sch (KiCad schematic (older format))
At the start: 1 part

Commit message: finishing schematic
Parts:
- gave numbers to parts that had none: 1
Changed lines of the file:
@@
 $Descr A4 11693 8268
 encoding utf-8
-Sheet 14 20
+Sheet 14 21
 Title ""
 Date ""
@@
 $EndDescr
 $Comp
-L atom:atom_G U?
+L atom:atom_G U15
 U 1 1 5DB8B498
 P 4600 3150
-F 0 "U?" H 6000 1467 60  0000 C CNN
+F 0 "U15" H 6000 1467 60  0000 C CNN
 F 1 "atom_G" H 6000 1361 60  0000 C CNN
 F 2 "" H 4750 3200 60  0001 R CNN

Commit message: first gbrs
Parts:
- U15: value atom_G -> atom_A_copy; footprint (none) -> Atom:FCBGA11702; symbol atom:atom_G -> atom:atom_A_copy
Changed lines of the file:
@@
 $EndDescr
 $Comp
-L atom:atom_G U15
-U 1 1 5DB8B498
+L atom:atom_A_copy U15
+U 7 1 5DB8B498
 P 4600 3150
 F 0 "U15" H 6000 1467 60  0000 C CNN
-F 1 "atom_G" H 6000 1361 60  0000 C CNN
-F 2 "" H 4750 3200 60  0001 R CNN
+F 1 "atom_A_copy" H 6000 1361 60  0000 C CNN
+F 2 "Atom:FCBGA11702" H 4750 3200 60  0001 R CNN
 F 3 "" H 4750 3000 60  0001 R CNN
-	1    4600 3150
+	7    4600 3150
 	1    0    0    -1
 $EndComp
