File: CPU_H.sch (KiCad schematic (older format))
At the start: 1 part

Commit message: finishing schematic
Parts:
- gave numbers to parts that had none: 1
Changed lines of the file:
@@
 $Descr A4 11693 8268
 encoding utf-8
-Sheet 15 20
+Sheet 15 21
 Title ""
 Date ""
@@
 $EndDescr
 $Comp
-L atom:atom_H U?
+L atom:atom_H U16
 U 1 1 5DB8CDAC
 P 4750 2700
-F 0 "U?" H 5950 3903 60  0000 C CNN
+F 0 "U16" H 5950 3903 60  0000 C CNN
 F 1 "atom_H" H 5950 3797 60  0000 C CNN
 F 2 "" H 4900 2750 60  0001 R CNN

Commit message: first gbrs
Parts:
- U16: value atom_H -> atom_A_copy; footprint (none) -> Atom:FCBGA11702; symbol atom:atom_H -> atom:atom_A_copy
Connections:
- net SOC_GPIO_S5_1: now reaches U16.B16 (GPIO_S5[01])
- net SOC_GPIO_S5_0: now reaches U16.B18 (GPIO_S5[00])
- net SOC_GPIO_S5_2: now reaches U16.C18 (GPIO_S5[02])
Changed lines of the file:
@@
 $EndDescr
 $Comp
-L atom:atom_H U16
-U 1 1 5DB8CDAC
-P 4750 2700
-F 0 "U16" H 5950 3903 60  0000 C CNN
-F 1 "atom_H" H 5950 3797 60  0000 C CNN
-F 2 "" H 4900 2750 60  0001 R CNN
-F 3 "" H 4900 2550 60  0001 R CNN
-	1    4750 2700
+L atom:atom_A_copy U16
+U 8 1 5DB8CDAC
+P 4750 2000
+F 0 "U16" H 5950 3203 60  0000 C CNN
+F 1 "atom_A_copy" H 5950 3097 60  0000 C CNN
+F 2 "Atom:FCBGA11702" H 4900 2050 60  0001 R CNN
+F 3 "" H 4900 1850 60  0001 R CNN
+	8    4750 2000
 	1    0    0    -1
 $EndComp
+Text GLabel 4750 3100 0    50   BiDi ~ 0
+SOC_GPIO_S5_0
+Text GLabel 4750 3000 0    50   BiDi ~ 0
+SOC_GPIO_S5_1
+Text GLabel 4750 3600 0    50   BiDi ~ 0
+SOC_GPIO_S5_2
 $EndSCHEMATC
