File: CPU_I.sch (KiCad schematic (older format))
At the start: 1 part

Commit message: finishing schematic
Parts:
- gave numbers to parts that had none: 1
Changed lines of the file:
@@
 $Descr A4 11693 8268
 encoding utf-8
-Sheet 16 20
+Sheet 16 21
 Title ""
 Date ""
@@
 $EndDescr
 $Comp
-L atom:atom_I U?
+L atom:atom_I U17
 U 1 1 5DB8E2A7
 P 4700 1900
-F 0 "U?" H 5850 2190 60  0000 C CNN
+F 0 "U17" H 5850 2190 60  0000 C CNN
 F 1 "atom_I" H 5850 2084 60  0000 C CNN
 F 2 "" H 4900 1950 60  0001 L CNN

Commit message: first gbrs
Parts:
- added R175, R176, R177, R178, R179, R180: 0Ohm, Resistor_SMD:R_0603_1608Metric, symbol Device:R_Small
- added R181: 10KOhm, Resistor_SMD:R_0603_1608Metric, symbol Device:R_Small
- added TP3: TestPoint, TestPoint:TestPoint_Pad_D2.0mm, symbol Connector:TestPoint
- U17: value atom_I -> atom_A_copy; footprint (none) -> Atom:FCBGA11702; symbol atom:atom_I -> atom:atom_A_copy
Connections:
- net at U17.A29 (RESERVED): now also R181.2
- net at U17.AH2 (RSVD_GND[3]): now also R175.1
- net at U17.AH3 (RSVD_GND[2]): now also R176.1
- net at U17.AM2 (RSVD_GND[1]): now also R177.1
- net at U17.AM3 (RSVD_GND[0]): now also R178.1
- net at U17.B30 (RESERVED): now also TP3.1
- net at U17.BB5 (RSVD_GND[6]): now also R179.1
- net at U17.BB7 (RSVD_GND[7]): now also R180.1
- new net GND: R175.2, R176.2, R177.2, R178.2, R179.2, R180.2, R181.1
Changed lines of the file:
@@
 $EndDescr
 $Comp
-L atom:atom_I U17
-U 1 1 5DB8E2A7
+L atom:atom_A_copy U17
+U 9 1 5DB8E2A7
 P 4700 1900
 F 0 "U17" H 5850 2190 60  0000 C CNN
-F 1 "atom_I" H 5850 2084 60  0000 C CNN
-F 2 "" H 4900 1950 60  0001 L CNN
+F 1 "atom_A_copy" H 5850 2084 60  0000 C CNN
+F 2 "Atom:FCBGA11702" H 4900 1950 60  0001 L CNN
 F 3 "" H 4900 1750 60  0001 L CNN
-	1    4700 1900
+	9    4700 1900
 	1    0    0    -1
 $EndComp
+$Comp
+L Device:R_Small R176
+U 1 1 5DD2D3AF
+P 5600 6000
+F 0 "R176" H 5659 6046 50  0000 L CNN
+F 1 "0Ohm" H 5659 5955 50  0000 L CNN
+F 2 "Resistor_SMD:R_0603_1608Metric" H 5600 6000 50  0001 C CNN
+F 3 "~" H 5600 6000 50  0001 C CNN
+	1    5600 6000
+	1    0    0    -1
+$EndComp
+$Comp
+L Device:R_Small R175
+U 1 1 5DD2D6E0
+P 5500 6000
+F 0 "R175" H 5559 6046 50  0000 L CNN
+F 1 "0Ohm" H 5559 5955 50  0000 L CNN
+F 2 "Resistor_SMD:R_0603_1608Metric" H 5500 6000 50  0001 C CNN
+F 3 "~" H 5500 6000 50  0001 C CNN
+	1    5500 6000
+	1    0    0    -1
+$EndComp
+$Comp
+L power:GND #PWR0343
+U 1 1 5DD2D9EA
+P 5500 6100
+F 0 "#PWR0343" H 5500 5850 50  0001 C CNN
+F 1 "GND" H 5505 5927 50  0000 C CNN
+F 2 "" H 5500 6100 50  0001 C CNN
+F 3 "" H 5500 6100 50  0001 C CNN
+	1    5500 6100
+	1    0    0    -1
+$EndComp
+$Comp
+L power:GND #PWR0344
+U 1 1 5DD2DBC2
+P 5600 6100
+F 0 "#PWR0344" H 5600 5850 50  0001 C CNN
+F 1 "GND" H 5605 5927 50  0000 C CNN
+F 2 "" H 5600 6100 50  0001 C CNN
+F 3 "" H 5600 6100 50  0001 C CNN
+	1    5600 6100
+	1    0    0    -1
+$EndComp
+$Comp
+L Device:R_Small R178
+U 1 1 5DD351B8
+P 5800 6000
+F 0 "R178" H 5859 6046 50  0000 L CNN
+F 1 "0Ohm" H 5859 5955 50  0000 L CNN
+F 2 "Resistor_SMD:R_0603_1608Metric" H 5800 6000 50  0001 C CNN
+F 3 "~" H 5800 6000 50  0001 C CNN
+	1    5800 6000
+	1    0    0    -1
+$EndComp
+$Comp
+L Device:R_Small R177
+U 1 1 5DD351BE
+P 5700 6000
+F 0 "R177" H 5759 6046 50  0000 L CNN
+F 1 "0Ohm" H 5759 5955 50  0000 L CNN
+F 2 "Resistor_SMD:R_0603_1608Metric" H 5700 6000 50  0001 C CNN
+F 3 "~" H 5700 6000 50  0001 C CNN
+	1    5700 6000
+	1    0    0    -1
+$EndComp
+$Comp
+L power:GND #PWR0345
+U 1 1 5DD351C4
+P 5700 6100
+F 0 "#PWR0345" H 5700 5850 50  0001 C CNN
+F 1 "GND" H 5705 5927 50  0000 C CNN
+F 2 "" H 5700 6100 50  0001 C CNN
+F 3 "" H 5700 6100 50  0001 C CNN
+	1    5700 6100
+	1    0    0    -1
+$EndComp
+$Comp
+L power:GND #PWR0346
+U 1 1 5DD351CA
+P 5800 6100
+F 0 "#PWR0346" H 5800 5850 50  0001 C CNN
+F 1 "GND" H 5805 5927 50  0000 C CNN
+F 2 "" H 5800 6100 50  0001 C CNN
+F 3 "" H 5800 6100 50  0001 C CNN
+	1    5800 6100
+	1    0    0    -1
+$EndComp
+$Comp
+L Device:R_Small R181
+U 1 1 5DD35752
+P 7100 4900
+F 0 "R181" V 6904 4900 50  0000 C CNN
+F 1 "10KOhm" V 6995 4900 50  0000 C CNN
+F 2 "Resistor_SMD:R_0603_1608Metric" H 7100 4900 50  0001 C CNN
+F 3 "~" H 7100 4900 50  0001 C CNN
+	1    7100 4900
+	0    1    1    0
+$EndComp
+$Comp
+L power:GND #PWR0347
+U 1 1 5DD35A3C
+P 7200 4900
+F 0 "#PWR0347" H 7200 4650 50  0001 C CNN
+F 1 "GND" V 7205 4772 50  0000 R CNN
+F 2 "" H 7200 4900 50  0001 C CNN
+F 3 "" H 7200 4900 50  0001 C CNN
+	1    7200 4900
+	0    -1   -1   0
+$EndComp
+$Comp
+L Connector:TestPoint TP3
+U 1 1 5DD36962
+P 7000 4800
+F 0 "TP3" V 6954 4988 50  0000 L CNN
+F 1 "TestPoint" V 7045 4988 50  0000 L CNN
+F 2 "TestPoint:TestPoint_Pad_D2.0mm" H 7200 4800 50  0001 C CNN
+F 3 "~" H 7200 4800 50  0001 C CNN
+	1    7000 4800
+	0    1    1    0
+$EndComp
+$Comp
+L power:GND #PWR0348
+U 1 1 5DD531F9
+P 5800 6100
+F 0 "#PWR0348" H 5800 5850 50  0001 C CNN
+F 1 "GND" H 5805 5927 50  0000 C CNN
+F 2 "" H 5800 6100 50  0001 C CNN
+F 3 "" H 5800 6100 50  0001 C CNN
+	1    5800 6100
+	1    0    0    -1
+$EndComp
+$Comp
+L Device:R_Small R180
+U 1 1 5DD531FF
+P 6000 6000
+F 0 "R180" H 6059 6046 50  0000 L CNN
+F 1 "0Ohm" H 6059 5955 50  0000 L CNN
+F 2 "Resistor_SMD:R_0603_1608Metric" H 6000 6000 50  0001 C CNN
+F 3 "~" H 6000 6000 50  0001 C CNN
+	1    6000 6000
+	1    0    0    -1
+$EndComp
+$Comp
+L Device:R_Small R179
+U 1 1 5DD53205
+P 5900 6000
+F 0 "R179" H 5959 6046 50  0000 L CNN
+F 1 "0Ohm" H 5959 5955 50  0000 L CNN
+F 2 "Resistor_SMD:R_0603_1608Metric" H 5900 6000 50  0001 C CNN
+F 3 "~" H 5900 6000 50  0001 C CNN
+	1    5900 6000
+	1    0    0    -1
+$EndComp
+$Comp
+L power:GND #PWR0349
+U 1 1 5DD5320B
+P 5900 6100
+F 0 "#PWR0349" H 5900 5850 50  0001 C CNN
+F 1 "GND" H 5905 5927 50  0000 C CNN
+F 2 "" H 5900 6100 50  0001 C CNN
+F 3 "" H 5900 6100 50  0001 C CNN
+	1    5900 6100
+	1    0    0    -1
+$EndComp
+$Comp
+L power:GND #PWR0350
+U 1 1 5DD53211
+P 6000 6100
+F 0 "#PWR0350" H 6000 5850 50  0001 C CNN
+F 1 "GND" H 6005 5927 50  0000 C CNN
+F 2 "" H 6000 6100 50  0001 C CNN
+F 3 "" H 6000 6100 50  0001 C CNN
+	1    6000 6100
+	1    0    0    -1
+$EndComp
