File: CPU_J.sch (KiCad schematic (older format))
At the start: 1 part

Commit message: finishing schematic
Parts:
- gave numbers to parts that had none: 1
Changed lines of the file:
@@
 $Descr A4 11693 8268
 encoding utf-8
-Sheet 17 20
+Sheet 17 21
 Title ""
 Date ""
@@
 $EndDescr
 $Comp
-L atom:atom_J U?
+L atom:atom_J U18
 U 1 1 5DB9065F
 P 4450 3100
-F 0 "U?" H 5600 1317 60  0000 C CNN
+F 0 "U18" H 5600 1317 60  0000 C CNN
 F 1 "atom_J" H 5600 1211 60  0000 C CNN
 F 2 "" H 4600 3150 60  0001 R CNN

Commit message: first gbrs
Parts:
- added C170: 0.1uF, Capacitor_SMD:C_0603_1608Metric, symbol Device:C_Small
- added R182: 2.2KOhm, Resistor_SMD:R_0603_1608Metric, symbol Device:R_Small
- added R183: 420Ohm, Resistor_SMD:R_0603_1608Metric, symbol Device:R_Small
- added U33: SN74LVC1G14DBVR, SN74LVC1G14DBVR:SN74LVC1G14DBVR, symbol SN74LVC1G14DBVR:SN74LVC1G14DBVR
- U18: value atom_J -> atom_A_copy; footprint (none) -> Atom:FCBGA11702; symbol atom:atom_J -> atom:atom_A_copy
Connections:
- net at U18.AK12 (DDI_RCOMP_P): now also R183.1
- net at U18.AK13 (DDI_RCOMP_N): now also R183.2
- net HDMI_CLK_DN: now reaches U18.AP2 (DDI0_TXN[3])
- net HDMI_CLK_DP: now reaches U18.AP3 (DDI0_TXP[3])
- net HDMI_TX0_DN: now reaches U18.AR1 (DDI0_TXN[2])
- net HDMI_TX0_DP: now reaches U18.AR3 (DDI0_TXP[2])
- net HDMI_TX1_DP: now reaches U18.AT2 (DDI0_TXP[1])
- net HDMI_TX1_DN: now reaches U18.AT3 (DDI0_TXN[1])
- net HDMI_TX2_DN: now reaches U18.AV2 (DDI0_TXN[0])
- net HDMI_TX2_DP: now reaches U18.AV3 (DDI0_TXP[0])
- net HDMI_DDCDAT: now reaches U18.C26 (DDI0_DDCDATA)
- net HDMI_DDCCLK: now reaches U18.C27 (DDI0_BKLTEN)
- net at U18.D27 (DDI0_HPD): now also U33.4 (Y)
- net GND: now reaches U18.G30 (DDI1_DDCCLK)
- net GND: now also U18.K30 (DDI1_HPD), C170.2, R182.1, U33.3 (GND)
- net at U18.P30 (DDI1_DDCDATA): now also R182.2
- new net +V1P8S: C170.1, U33.5 (VCC)
- new net HDMI_HPD: U33.2 (A)
Changed lines of the file:
@@
 $EndDescr
 $Comp
-L atom:atom_J U18
-U 1 1 5DB9065F
-P 4450 3100
-F 0 "U18" H 5600 1317 60  0000 C CNN
-F 1 "atom_J" H 5600 1211 60  0000 C CNN
-F 2 "" H 4600 3150 60  0001 R CNN
-F 3 "" H 4600 2950 60  0001 R CNN
-	1    4450 3100
+L atom:atom_A_copy U18
+U 10 1 5DB9065F
+P 4450 2400
+F 0 "U18" H 5600 617 60  0000 C CNN
+F 1 "atom_A_copy" H 5600 511 60  0000 C CNN
+F 2 "Atom:FCBGA11702" H 4600 2450 60  0001 R CNN
+F 3 "" H 4600 2250 60  0001 R CNN
+	10   4450 2400
 	1    0    0    -1
 $EndComp
+$Comp
+L power:GND #PWR0351
+U 1 1 5DD2C697
+P 6750 3400
+F 0 "#PWR0351" H 6750 3150 50  0001 C CNN
+F 1 "GND" V 6755 3272 50  0000 R CNN
+F 2 "" H 6750 3400 50  0001 C CNN
+F 3 "" H 6750 3400 50  0001 C CNN
+	1    6750 3400
+	0    -1   -1   0
+$EndComp
+$Comp
+L Device:R_Small R182
+U 1 1 5DD2C957
+P 6850 3100
+F 0 "R182" V 6654 3100 50  0000 C CNN
+F 1 "2.2KOhm" V 6745 3100 50  0000 C CNN
+F 2 "Resistor_SMD:R_0603_1608Metric" H 6850 3100 50  0001 C CNN
+F 3 "~" H 6850 3100 50  0001 C CNN
+	1    6850 3100
+	0    1    1    0
+$EndComp
+$Comp
+L power:GND #PWR0352
+U 1 1 5DD2CCAD
+P 6950 3100
+F 0 "#PWR0352" H 6950 2850 50  0001 C CNN
+F 1 "GND" V 6955 2972 50  0000 R CNN
+F 2 "" H 6950 3100 50  0001 C CNN
+F 3 "" H 6950 3100 50  0001 C CNN
+	1    6950 3100
+	0    -1   -1   0
+$EndComp
+$Comp
+L power:GND #PWR0353
+U 1 1 5DD2CFEB
+P 6750 3500
+F 0 "#PWR0353" H 6750 3250 50  0001 C CNN
+F 1 "GND" V 6755 3372 50  0000 R CNN
+F 2 "" H 6750 3500 50  0001 C CNN
+F 3 "" H 6750 3500 50  0001 C CNN
+	1    6750 3500
+	0    -1   -1   0
+$EndComp
+Text GLabel 4450 4000 0    50   Output ~ 0
+HDMI_TX2_DP
+Text GLabel 4450 3900 0    50   Output ~ 0
+HDMI_TX2_DN
+Text GLabel 4450 3700 0    50   Output ~ 0
+HDMI_TX1_DP
+Text GLabel 4450 3800 0    50   Output ~ 0
+HDMI_TX1_DN
+Text GLabel 4450 3600 0    50   Output ~ 0
+HDMI_TX0_DP
+Text GLabel 4450 3500 0    50   Output ~ 0
+HDMI_TX0_DN
+Text GLabel 4450 3400 0    50   Output ~ 0
+HDMI_CLK_DP
+Text GLabel 4450 3300 0    50   Output ~ 0
+HDMI_CLK_DN
+Text GLabel 4450 4300 0    50   BiDi ~ 0
+HDMI_DDCDAT
+Text GLabel 4450 4400 0    50   Output ~ 0
+HDMI_DDCCLK
+$Comp
+L Device:R_Small R183
+U 1 1 5DD32BE7
+P 6850 3600
+F 0 "R183" V 6654 3600 50  0000 C CNN
+F 1 "420Ohm" V 6745 3600 50  0000 C CNN
+F 2 "Resistor_SMD:R_0603_1608Metric" H 6850 3600 50  0001 C CNN
+F 3 "~" H 6850 3600 50  0001 C CNN
+	1    6850 3600
+	0    1    1    0
+$EndComp
+Wire Wire Line
+	6750 3700 7100 3700
+Wire Wire Line
+	7100 3700 7100 3600
+Wire Wire Line
+	7100 3600 6950 3600
+$Comp
+L SN74LVC1G14DBVR:SN74LVC1G14DBVR U33
+U 1 1 5DD3AD54
+P 900 4500
+F 0 "U33" H 2000 4887 60  0000 C CNN
+F 1 "SN74LVC1G14DBVR" H 2000 4781 60  0000 C CNN
+F 2 "SN74LVC1G14DBVR:SN74LVC1G14DBVR" H 2000 4740 60  0001 C CNN
+F 3 "" H 900 4500 60  0000 C CNN
+	1    900  4500
+	1    0    0    -1
+$EndComp
+Text GLabel 900  4600 0    50   Input ~ 0
+HDMI_HPD
+$Comp
+L power:GND #PWR0354
+U 1 1 5DD3BE82
+P 3100 4700
+F 0 "#PWR0354" H 3100 4450 50  0001 C CNN
+F 1 "GND" V 3105 4572 50  0000 R CNN
+F 2 "" H 3100 4700 50  0001 C CNN
+F 3 "" H 3100 4700 50  0001 C CNN
+	1    3100 4700
+	0    -1   -1   0
+$EndComp
+Wire Wire Line
+	4450 4600 3100 4600
+$Comp
+L POWER:+V1P8S #PWR0355
+U 1 1 5DD3D2AF
+P 3100 3800
+F 0 "#PWR0355" H 3100 3650 50  0001 C CNN
+F 1 "+V1P8S" H 3117 3973 50  0000 C CNN
+F 2 "" H 3100 3800 50  0001 C CNN
+F 3 "" H 3100 3800 50  0001 C CNN
+	1    3100 3800
+	1    0    0    -1
+$EndComp
+$Comp
+L Device:C_Small C170
+U 1 1 5DD3D4CB
+P 2800 3900
+F 0 "C170" V 2571 3900 50  0000 C CNN
+F 1 "0.1uF" V 2662 3900 50  0000 C CNN
+F 2 "Capacitor_SMD:C_0603_1608Metric" H 2800 3900 50  0001 C CNN
+F 3 "~" H 2800 3900 50  0001 C CNN
+	1    2800 3900
+	0    1    1    0
+$EndComp
+$Comp
+L power:GND #PWR0356
+U 1 1 5DD3D8A3
+P 2700 3900
+F 0 "#PWR0356" H 2700 3650 50  0001 C CNN
+F 1 "GND" V 2705 3772 50  0000 R CNN
+F 2 "" H 2700 3900 50  0001 C CNN
+F 3 "" H 2700 3900 50  0001 C CNN
+	1    2700 3900
+	0    1    1    0
+$EndComp
+Wire Wire Line
+	3100 3800 3100 3900
+Wire Wire Line
+	2900 3900 3100 3900
+Connection ~ 3100 3900
+Wire Wire Line
+	3100 3900 3100 4500
 $EndSCHEMATC
