File: CPU_K.sch (KiCad schematic (older format))
At the start: 1 part

Commit message: finishing schematic
Parts:
- gave numbers to parts that had none: 1
Changed lines of the file:
@@
 $Descr A4 11693 8268
 encoding utf-8
-Sheet 18 20
+Sheet 18 21
 Title ""
 Date ""
@@
 $EndDescr
 $Comp
-L atom:atom_K U?
+L atom:atom_K U19
 U 1 1 5DB91C36
 P 4650 2700
-F 0 "U?" H 5650 2990 60  0000 C CNN
+F 0 "U19" H 5650 2990 60  0000 C CNN
 F 1 "atom_K" H 5650 2884 60  0000 C CNN
 F 2 "" H 4850 2750 60  0001 L CNN

Commit message: first gbrs
Parts:
- U19: value atom_K -> atom_A_copy; footprint (none) -> Atom:FCBGA11702; symbol atom:atom_K -> atom:atom_A_copy
Changed lines of the file:
@@
 $EndDescr
 $Comp
-L atom:atom_K U19
-U 1 1 5DB91C36
+L atom:atom_A_copy U19
+U 11 1 5DB91C36
 P 4650 2700
 F 0 "U19" H 5650 2990 60  0000 C CNN
-F 1 "atom_K" H 5650 2884 60  0000 C CNN
-F 2 "" H 4850 2750 60  0001 L CNN
+F 1 "atom_A_copy" H 5650 2884 60  0000 C CNN
+F 2 "Atom:FCBGA11702" H 4850 2750 60  0001 L CNN
 F 3 "" H 4850 2550 60  0001 L CNN
-	1    4650 2700
+	11   4650 2700
 	1    0    0    -1
 $EndComp
