File: CPU_L.sch (KiCad schematic (older format))
At the start: 1 part

Commit message: finishing schematic
Parts:
- gave numbers to parts that had none: 1
Changed lines of the file:
@@
 $Descr A4 11693 8268
 encoding utf-8
-Sheet 19 20
+Sheet 19 21
 Title ""
 Date ""
@@
 $EndDescr
 $Comp
-L atom:atom_L U?
+L atom:atom_L U20
 U 1 1 5DB931DD
 P 5100 3200
-F 0 "U?" H 6050 3490 60  0000 C CNN
+F 0 "U20" H 6050 3490 60  0000 C CNN
 F 1 "atom_L" H 6050 3384 60  0000 C CNN
 F 2 "" H 5300 3250 60  0001 L CNN

Commit message: first gbrs
Parts:
- added R184: 150Ohm, Resistor_SMD:R_0603_1608Metric, symbol Device:R_Small
- U20: footprint (none) -> Atom:FCBGA11702; symbol atom:atom_L -> atom:atom_A_copy
Connections:
- net at U20.P14 (MCSI_RCOMP): now also R184.1
- new net GND: R184.2
Changed lines of the file:
@@
 $EndDescr
 $Comp
-L atom:atom_L U20
-U 1 1 5DB931DD
+L atom:atom_A_copy U20
+U 12 1 5DB931DD
 P 5100 3200
 F 0 "U20" H 6050 3490 60  0000 C CNN
 F 1 "atom_L" H 6050 3384 60  0000 C CNN
-F 2 "" H 5300 3250 60  0001 L CNN
+F 2 "Atom:FCBGA11702" H 5300 3250 60  0001 L CNN
 F 3 "" H 5300 3050 60  0001 L CNN
-	1    5100 3200
+	12   5100 3200
 	1    0    0    -1
 $EndComp
+$Comp
+L Device:R_Small R184
+U 1 1 5DD31888
+P 7100 3400
+F 0 "R184" V 7296 3400 50  0000 C CNN
+F 1 "150Ohm" V 7205 3400 50  0000 C CNN
+F 2 "Resistor_SMD:R_0603_1608Metric" H 7100 3400 50  0001 C CNN
+F 3 "~" H 7100 3400 50  0001 C CNN
+	1    7100 3400
+	0    -1   -1   0
+$EndComp
+$Comp
+L power:GND #PWR0357
+U 1 1 5DD31DD3
+P 7200 3400
+F 0 "#PWR0357" H 7200 3150 50  0001 C CNN
+F 1 "GND" V 7205 3272 50  0000 R CNN
+F 2 "" H 7200 3400 50  0001 C CNN
+F 3 "" H 7200 3400 50  0001 C CNN
+	1    7200 3400
+	0    -1   -1   0
+$EndComp
 $EndSCHEMATC
