File: YellowCake.kicad_pcb (KiCad board)
At the start: 4 copper layers, 95.9 x 90.2 mm, 400 parts, among them J1 10029449-111RLF, J2 USB_A, J3 USB3_A, J4 SODIMM-200, J5 Micro_SD_Card, J6 Conn_Coaxial_Power, J7 Conn_01x08_Male, Q1 2N7002K, Q2 2N7002K, Q3 MMBT3904, Q4 2N7002K, Q5 2N7002K, Q6 2N7002K, Q7 MBT3904DW1, Q8 MBT3904DW1, Q9 BSS138, SW1 SW_Push, U1 CS4207-CNZ, U2 ISL95837HRZ-T, U21 NB670, U22 IRF9321, U23 NCT3012S, U24 TXS0104EYZTR, U25 APL5912KAC, U26 FDMS7602S, U27 FDMS7602S, U28 APL5933, U29 APL5933, U3 TPD12S016PWR, U30 NCP606MN18T2G, U31 TS3A27518ERTWR, U32 25LCxxx, U4 TPD4S012DRYR, U5 TPS2066DR, U6 TPD4EUSB30, U7 TPD4S012DRYR, U8 TPD6E001RSER

Commit message: first gbrs
Parts:
- removed FCBGA1170: VAL**, Atom:FCBGA11702
- removed H1, H2, H3, H4: MountingHole_Pad, MountingHole:MountingHole_3.2mm_M3_Pad
- added C168: 18pF, Capacitor_SMD:C_0603_1608Metric, F.Cu at (184.9, 45.6)
- added C169: 18pF, Capacitor_SMD:C_0603_1608Metric, F.Cu at (180.9, 43.1)
- added C170: 0.1uF, Capacitor_SMD:C_0603_1608Metric, F.Cu at (172.8, 57.4)
- added C171: 27pF, Capacitor_SMD:C_0603_1608Metric, F.Cu at (136.4, 54.8)
- added C172: 10pF, Capacitor_SMD:C_0603_1608Metric, F.Cu at (141.5, 53.1)
- added C173: 27pF, Capacitor_SMD:C_0603_1608Metric, F.Cu at (141.5, 61.1)
- added JP2: Jumper, Jumper:SolderJumper-2_P1.3mm_Open_RoundedPad1.0x1.5mm, F.Cu at (135.3, 46.6)
- added R159: 10KOhm, Resistor_SMD:R_0603_1608Metric, F.Cu at (176.9, 47.1)
- added R160: 402Ohm, Resistor_SMD:R_0603_1608Metric, F.Cu at (172.8, 50.5)
- added R161: 10KOhm, Resistor_SMD:R_0603_1608Metric, F.Cu at (181.9, 40.6)
- added R162: 1KOhm, Resistor_SMD:R_0603_1608Metric, F.Cu at (168.8, 48.0)
- added R163: 10KOhm, Resistor_SMD:R_0603_1608Metric, F.Cu at (176.9, 44.6)
- added R164: 10KOhm, Resistor_SMD:R_0603_1608Metric, F.Cu at (177.9, 40.6)
- added R165: 10KOhm, Resistor_SMD:R_0603_1608Metric, F.Cu at (168.8, 50.5)
- added R166: 0Ohm, Resistor_SMD:R_0603_1608Metric, F.Cu at (186.0, 40.6)
- added R167: 73.2Ohm, Resistor_SMD:R_0603_1608Metric, F.Cu at (172.8, 48.0)
- added R168: 49.9Ohm, Resistor_SMD:R_0603_1608Metric, F.Cu at (180.9, 45.6)
- added R169: 49.9Ohm, Resistor_SMD:R_0603_1608Metric, F.Cu at (176.9, 49.7)
- added R170: 150Ohm, Resistor_SMD:R_0603_1608Metric, F.Cu at (184.9, 43.1)
- added R171: 150Ohm, Resistor_SMD:R_0603_1608Metric, F.Cu at (180.9, 48.1)
- added R172: 49.9Ohm, Resistor_SMD:R_0603_1608Metric, F.Cu at (172.9, 44.6)
- added R173: 357Ohm, Resistor_SMD:R_0603_1608Metric, F.Cu at (188.9, 43.1)
- added R174: 10MOhm, Resistor_SMD:R_0603_1608Metric, F.Cu at (180.9, 50.6)
- added R175: 0Ohm, Resistor_SMD:R_0603_1608Metric, B.Cu at (108.9, 50.6)
- added R176: 0Ohm, Resistor_SMD:R_0603_1608Metric, B.Cu at (104.9, 54.7)
- added R177: 0Ohm, Resistor_SMD:R_0603_1608Metric, B.Cu at (111.4, 50.6)
- added R178: 0Ohm, Resistor_SMD:R_0603_1608Metric, B.Cu at (108.9, 54.6)
- added R179: 0Ohm, Resistor_SMD:R_0603_1608Metric, B.Cu at (104.9, 58.7)
- added R180: 0Ohm, Resistor_SMD:R_0603_1608Metric, B.Cu at (111.4, 54.6)
- added R181: 10KOhm, Resistor_SMD:R_0603_1608Metric, B.Cu at (107.4, 58.6)
- added R182: 2.2KOhm, Resistor_SMD:R_0603_1608Metric, F.Cu at (168.8, 57.4)
- added R183: 420Ohm, Resistor_SMD:R_0603_1608Metric, F.Cu at (168.8, 59.9)
- added R184: 150Ohm, Resistor_SMD:R_0603_1608Metric, B.Cu at (117.2, 50.6)
- added R185: 4.02KOhm, Resistor_SMD:R_0603_1608Metric, F.Cu at (139.0, 61.1)
- added R186: 47.5Ohm, Resistor_SMD:R_0603_1608Metric, F.Cu at (133.3, 50.8)
- added R187: 0Ohm, Resistor_SMD:R_0603_1608Metric, F.Cu at (133.9, 54.8)
- added R188: 0Ohm, Resistor_SMD:R_0603_1608Metric, F.Cu at (139.0, 57.1)
- added R189: 0Ohm, Resistor_SMD:R_0603_1608Metric, F.Cu at (141.5, 57.1)
- added R190: 0Ohm, Resistor_SMD:R_0603_1608Metric, F.Cu at (135.8, 50.8)
- added R191: 1MOhm, Resistor_SMD:R_0603_1608Metric, F.Cu at (139.0, 53.1)
- added TP1: TestPoint, TestPoint:TestPoint_Pad_D2.0mm, F.Cu at (173.9, 41.4)
- added TP2: TestPoint, TestPoint:TestPoint_Pad_D2.0mm, F.Cu at (168.9, 44.7)
- added TP3: TestPoint, TestPoint:TestPoint_Pad_D2.0mm, F.Cu at (104.3, 50.4)
- added U10, U11, U12, U13, U14, U15, U16, U17, U18, U19, U9: atom_A_copy, Atom:FCBGA11702, F.Cu at (149.3, 78.2)
- added U20: atom_L, Atom:FCBGA11702, F.Cu at (149.3, 78.2)
- added U33: SN74LVC1G14DBVR, SN74LVC1G14DBVR:SN74LVC1G14DBVR, F.Cu at (105.8, 64.2)
- added Y1: Crystal, Crystal:Crystal_SMD_3215-2Pin_3.2x1.5mm, F.Cu at (169.4, 41.0)
- added Y2: Crystal_GND24_Small, Crystal:Crystal_SMD_3225-4Pin_3.2x2.5mm_HandSoldering, F.Cu at (139.9, 47.7)
- C100, C101, C102, C103, C104, C105, C106, C107, C108, C109, C110, C111, C112, C113, C114, C115, C116, C117, C118, C119, C134, C135, C136, C51, C96, C97, C98, C99, D4, D5, D6, D7, D8, J1, J4, JP1, L16, L2, Q1, Q2, Q3, Q4, Q5, Q6, Q7, Q8, R100, R101, R102, R103, R111, R112, R113, R114, R115, R116, R117, R118, R119, R120, R121, R122, R123, R124, R125, R126, R127, R63, R64, R69, R92, R93, R94, R95, R96, R97, R98, R99, U25, U3: moved to B.Cu
- C50, R59, R60, R61, R62, R65, R66, R67, R68: moved to F.Cu
- moved R136 264.9 mm to (114.3, 40.3), turned to 90 degrees
- moved R137 262.4 mm to (116.8, 41.5), turned to 90 degrees
- moved C143 261.5 mm to (119.3, 41.5), turned to 90 degrees
- moved R135 261.5 mm to (111.8, 43.5), turned to 90 degrees
- moved R128 259.5 mm to (114.3, 44.3), turned to 90 degrees
- moved C122 258.1 mm to (121.8, 43.4), turned to 90 degrees
- moved C145 257.4 mm to (124.4, 43.4), turned to 90 degrees
- moved R130 256.9 mm to (116.8, 45.5), turned to 90 degrees
- moved L17 256.0 mm to (111.8, 47.5), turned to 90 degrees
- moved R133 256.0 mm to (119.3, 45.5), turned to 90 degrees
- moved C141 254.0 mm to (114.3, 48.3), turned to 90 degrees
- moved R139 252.4 mm to (122.4, 47.4), turned to 90 degrees
- moved C120 251.7 mm to (124.9, 47.4), turned to 90 degrees
- moved C142 251.2 mm to (117.4, 49.5), turned to 90 degrees
- moved C123 251.1 mm to (127.4, 47.3), turned to 90 degrees
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Routing:
- net (no net): track 76.0 -> 0.00 mm, vias 140 -> 0
